File: hardware/fpga-ice40/FPGA_Power.sch (KiCad schematic (older format))
At the start: 25 parts, among them U1 iCE40HX4K-TQ144

Commit message: Reannotate schematic symbols
Parts:
- renumbered C31 to C23, C32 to C24, C1 to C25, C2 to C26, C3 to C27, C4 to C28, C5 to C30, C6 to C31, C27 to C32, C7 to C33, C8 to C34, C9 to C35, C10 to C36, C11 to C37, C12 to C38, C13 to C39, C14 to C40, C28 to C41, C25 to C42, C26 to C43, R11 to R6, R12 to R7
Changed lines of the file:
@@
 $Descr USLetter 11000 8500
 encoding utf-8
-Sheet 3 12
+Sheet 10 12
 Title "Ferk-Cart iCE40 Devboard"
 Date "2020-06-29"
@@
 P 5200 3650
 AR Path="/5F56D89A" Ref="C?"  Part="1"
-AR Path="/5F35C9AC/5F56D89A" Ref="C1"  Part="1"
-F 0 "C1" H 5250 3750 50  0000 L CNN
+AR Path="/5F35C9AC/5F56D89A" Ref="C25"  Part="1"
+F 0 "C25" H 5250 3750 50  0000 L CNN
 F 1 "100n" H 5250 3550 50  0000 L CNN
 F 2 "Capacitor_SMD:C_0603_1608Metric" H 5238 3500 50  0001 C CNN
@@
 P 5500 3650
 AR Path="/5F56D8A0" Ref="C?"  Part="1"
-AR Path="/5F35C9AC/5F56D8A0" Ref="C2"  Part="1"
-F 0 "C2" H 5550 3750 50  0000 L CNN
+AR Path="/5F35C9AC/5F56D8A0" Ref="C26"  Part="1"
+F 0 "C26" H 5550 3750 50  0000 L CNN
 F 1 "100n" H 5550 3550 50  0000 L CNN
 F 2 "Capacitor_SMD:C_0603_1608Metric" H 5538 3500 50  0001 C CNN
@@
 P 5800 3650
 AR Path="/5F56D8A6" Ref="C?"  Part="1"
-AR Path="/5F35C9AC/5F56D8A6" Ref="C3"  Part="1"
-F 0 "C3" H 5850 3750 50  0000 L CNN
+AR Path="/5F35C9AC/5F56D8A6" Ref="C27"  Part="1"
+F 0 "C27" H 5850 3750 50  0000 L CNN
 F 1 "100n" H 5850 3550 50  0000 L CNN
 F 2 "Capacitor_SMD:C_0603_1608Metric" H 5838 3500 50  0001 C CNN
@@
 P 6100 3650
 AR Path="/5F56D8B8" Ref="C?"  Part="1"
-AR Path="/5F35C9AC/5F56D8B8" Ref="C4"  Part="1"
-F 0 "C4" H 6150 3750 50  0000 L CNN
+AR Path="/5F35C9AC/5F56D8B8" Ref="C28"  Part="1"
+F 0 "C28" H 6150 3750 50  0000 L CNN
 F 1 "100n" H 6150 3550 50  0000 L CNN
 F 2 "Capacitor_SMD:C_0603_1608Metric" H 6138 3500 50  0001 C CNN
@@
 P 8850 3650
 AR Path="/5F56D8C4" Ref="C?"  Part="1"
-AR Path="/5F35C9AC/5F56D8C4" Ref="C5"  Part="1"
-F 0 "C5" H 8900 3750 50  0000 L CNN
+AR Path="/5F35C9AC/5F56D8C4" Ref="C30"  Part="1"
+F 0 "C30" H 8900 3750 50  0000 L CNN
 F 1 "10u" H 8900 3550 50  0000 L CNN
 F 2 "Capacitor_SMD:C_0603_1608Metric" H 8888 3500 50  0001 C CNN
@@
 P 9150 3650
 AR Path="/5F56D8CA" Ref="C?"  Part="1"
-AR Path="/5F35C9AC/5F56D8CA" Ref="C6"  Part="1"
-F 0 "C6" H 9200 3750 50  0000 L CNN
+AR Path="/5F35C9AC/5F56D8CA" Ref="C31"  Part="1"
+F 0 "C31" H 9200 3750 50  0000 L CNN
 F 1 "100n" H 9200 3550 50  0000 L CNN
 F 2 "Capacitor_SMD:C_0603_1608Metric" H 9188 3500 50  0001 C CNN
@@
 P 5500 4700
 AR Path="/5F56D8D6" Ref="C?"  Part="1"
-AR Path="/5F35C9AC/5F56D8D6" Ref="C9"  Part="1"
-F 0 "C9" H 5550 4800 50  0000 L CNN
+AR Path="/5F35C9AC/5F56D8D6" Ref="C35"  Part="1"
+F 0 "C35" H 5550 4800 50  0000 L CNN
 F 1 "100n" H 5550 4600 50  0000 L CNN
 F 2 "Capacitor_SMD:C_0603_1608Metric" H 5538 4550 50  0001 C CNN
@@
 P 5800 4700
 AR Path="/5F56D8DC" Ref="C?"  Part="1"
-AR Path="/5F35C9AC/5F56D8DC" Ref="C10"  Part="1"
-F 0 "C10" H 5850 4800 50  0000 L CNN
+AR Path="/5F35C9AC/5F56D8DC" Ref="C36"  Part="1"
+F 0 "C36" H 5850 4800 50  0000 L CNN
 F 1 "100n" H 5850 4600 50  0000 L CNN
 F 2 "Capacitor_SMD:C_0603_1608Metric" H 5838 4550 50  0001 C CNN
@@
 P 8850 4700
 AR Path="/5F56D8EF" Ref="C?"  Part="1"
-AR Path="/5F35C9AC/5F56D8EF" Ref="C25"  Part="1"
-F 0 "C25" H 8900 4800 50  0000 L CNN
+AR Path="/5F35C9AC/5F56D8EF" Ref="C42"  Part="1"
+F 0 "C42" H 8900 4800 50  0000 L CNN
 F 1 "10u" H 8900 4600 50  0000 L CNN
 F 2 "Capacitor_SMD:C_0603_1608Metric" H 8888 4550 50  0001 C CNN
@@
 P 9150 4700
 AR Path="/5F56D8F5" Ref="C?"  Part="1"
-AR Path="/5F35C9AC/5F56D8F5" Ref="C26"  Part="1"
-F 0 "C26" H 9200 4800 50  0000 L CNN
+AR Path="/5F35C9AC/5F56D8F5" Ref="C43"  Part="1"
+F 0 "C43" H 9200 4800 50  0000 L CNN
 F 1 "100n" H 9200 4600 50  0000 L CNN
 F 2 "Capacitor_SMD:C_0603_1608Metric" H 9188 4550 50  0001 C CNN
@@
 P 8600 4450
 AR Path="/5F56D905" Ref="R?"  Part="1"
-AR Path="/5F35C9AC/5F56D905" Ref="R12"  Part="1"
-F 0 "R12" V 8400 4450 50  0000 C CNN
+AR Path="/5F35C9AC/5F56D905" Ref="R7"  Part="1"
+F 0 "R7" V 8400 4450 50  0000 C CNN
 F 1 "100R" V 8500 4450 50  0000 C CNN
 F 2 "Resistor_SMD:R_0603_1608Metric" V 8530 4450 50  0001 C CNN
@@
 P 8600 3400
 AR Path="/5F56D90B" Ref="R?"  Part="1"
-AR Path="/5F35C9AC/5F56D90B" Ref="R11"  Part="1"
-F 0 "R11" V 8400 3400 50  0000 C CNN
+AR Path="/5F35C9AC/5F56D90B" Ref="R6"  Part="1"
+F 0 "R6" V 8400 3400 50  0000 C CNN
 F 1 "100R" V 8500 3400 50  0000 C CNN
 F 2 "Resistor_SMD:R_0603_1608Metric" V 8530 3400 50  0001 C CNN
@@
 P 4600 3650
 AR Path="/5F56D914" Ref="C?"  Part="1"
-AR Path="/5F35C9AC/5F56D914" Ref="C31"  Part="1"
-F 0 "C31" H 4650 3750 50  0000 L CNN
+AR Path="/5F35C9AC/5F56D914" Ref="C23"  Part="1"
+F 0 "C23" H 4650 3750 50  0000 L CNN
 F 1 "10u" H 4650 3550 50  0000 L CNN
 F 2 "Capacitor_SMD:C_0603_1608Metric" H 4638 3500 50  0001 C CNN
@@
 P 4900 3650
 AR Path="/5F56D91A" Ref="C?"  Part="1"
-AR Path="/5F35C9AC/5F56D91A" Ref="C32"  Part="1"
-F 0 "C32" H 4950 3750 50  0000 L CNN
+AR Path="/5F35C9AC/5F56D91A" Ref="C24"  Part="1"
+F 0 "C24" H 4950 3750 50  0000 L CNN
 F 1 "1u" H 4950 3550 50  0000 L CNN
 F 2 "Capacitor_SMD:C_0603_1608Metric" H 4938 3500 50  0001 C CNN
@@
 P 5200 4700
 AR Path="/5F56D947" Ref="C?"  Part="1"
-AR Path="/5F35C9AC/5F56D947" Ref="C8"  Part="1"
-F 0 "C8" H 5250 4800 50  0000 L CNN
+AR Path="/5F35C9AC/5F56D947" Ref="C34"  Part="1"
+F 0 "C34" H 5250 4800 50  0000 L CNN
 F 1 "100n" H 5250 4600 50  0000 L CNN
 F 2 "Capacitor_SMD:C_0603_1608Metric" H 5238 4550 50  0001 C CNN
@@
 P 4900 4700
 AR Path="/5F56D94D" Ref="C?"  Part="1"
-AR Path="/5F35C9AC/5F56D94D" Ref="C7"  Part="1"
-F 0 "C7" H 4950 4800 50  0000 L CNN
+AR Path="/5F35C9AC/5F56D94D" Ref="C33"  Part="1"
+F 0 "C33" H 4950 4800 50  0000 L CNN
 F 1 "100n" H 4950 4600 50  0000 L CNN
 F 2 "Capacitor_SMD:C_0603_1608Metric" H 4938 4550 50  0001 C CNN
@@
 P 3500 4400
 AR Path="/5F56D955" Ref="#PWR?"  Part="1"
-AR Path="/5F35C9AC/5F56D955" Ref="#PWR0129"  Part="1"
-F 0 "#PWR0129" H 3500 4150 50  0001 C CNN
+AR Path="/5F35C9AC/5F56D955" Ref="#PWR029"  Part="1"
+F 0 "#PWR029" H 3500 4150 50  0001 C CNN
 F 1 "GND" V 3504 4320 50  0000 R CNN
 F 2 "" H 3400 4050 50  0001 C CNN
@@
 P 7000 4700
 AR Path="/5F56D96B" Ref="C?"  Part="1"
-AR Path="/5F35C9AC/5F56D96B" Ref="C14"  Part="1"
-F 0 "C14" H 7050 4800 50  0000 L CNN
+AR Path="/5F35C9AC/5F56D96B" Ref="C40"  Part="1"
+F 0 "C40" H 7050 4800 50  0000 L CNN
 F 1 "100n" H 7050 4600 50  0000 L CNN
 F 2 "Capacitor_SMD:C_0603_1608Metric" H 7038 4550 50  0001 C CNN
@@
 P 6700 4700
 AR Path="/5F56D971" Ref="C?"  Part="1"
-AR Path="/5F35C9AC/5F56D971" Ref="C13"  Part="1"
-F 0 "C13" H 6750 4800 50  0000 L CNN
+AR Path="/5F35C9AC/5F56D971" Ref="C39"  Part="1"
+F 0 "C39" H 6750 4800 50  0000 L CNN
 F 1 "100n" H 6750 4600 50  0000 L CNN
 F 2 "Capacitor_SMD:C_0603_1608Metric" H 6738 4550 50  0001 C CNN
@@
 P 6400 4700
 AR Path="/5F56D97B" Ref="C?"  Part="1"
-AR Path="/5F35C9AC/5F56D97B" Ref="C12"  Part="1"
-F 0 "C12" H 6450 4800 50  0000 L CNN
+AR Path="/5F35C9AC/5F56D97B" Ref="C38"  Part="1"
+F 0 "C38" H 6450 4800 50  0000 L CNN
 F 1 "100n" H 6450 4600 50  0000 L CNN
 F 2 "Capacitor_SMD:C_0603_1608Metric" H 6438 4550 50  0001 C CNN
@@
 P 6100 4700
 AR Path="/5F56D981" Ref="C?"  Part="1"
-AR Path="/5F35C9AC/5F56D981" Ref="C11"  Part="1"
-F 0 "C11" H 6150 4800 50  0000 L CNN
+AR Path="/5F35C9AC/5F56D981" Ref="C37"  Part="1"
+F 0 "C37" H 6150 4800 50  0000 L CNN
 F 1 "100n" H 6150 4600 50  0000 L CNN
 F 2 "Capacitor_SMD:C_0603_1608Metric" H 6138 4550 50  0001 C CNN
@@
 P 4600 4700
 AR Path="/5F56D999" Ref="C?"  Part="1"
-AR Path="/5F35C9AC/5F56D999" Ref="C27"  Part="1"
-F 0 "C27" H 4650 4800 50  0000 L CNN
+AR Path="/5F35C9AC/5F56D999" Ref="C32"  Part="1"
+F 0 "C32" H 4650 4800 50  0000 L CNN
 F 1 "10u" H 4650 4600 50  0000 L CNN
 F 2 "Capacitor_SMD:C_0805_2012Metric" H 4638 4550 50  0001 C CNN
@@
 P 7300 4700
 AR Path="/5F56D9AA" Ref="C?"  Part="1"
-AR Path="/5F35C9AC/5F56D9AA" Ref="C28"  Part="1"
-F 0 "C28" H 7350 4800 50  0000 L CNN
+AR Path="/5F35C9AC/5F56D9AA" Ref="C41"  Part="1"
+F 0 "C41" H 7350 4800 50  0000 L CNN
 F 1 "100n" H 7350 4600 50  0000 L CNN
 F 2 "Capacitor_SMD:C_0603_1608Metric" H 7338 4550 50  0001 C CNN
@@
 P 7300 3900
 AR Path="/5F56D9C6" Ref="#PWR?"  Part="1"
-AR Path="/5F35C9AC/5F56D9C6" Ref="#PWR0130"  Part="1"
-F 0 "#PWR0130" H 7300 3650 50  0001 C CNN
+AR Path="/5F35C9AC/5F56D9C6" Ref="#PWR027"  Part="1"
+F 0 "#PWR027" H 7300 3650 50  0001 C CNN
 F 1 "GND" H 7303 3774 50  0000 C CNN
 F 2 "" H 7200 3550 50  0001 C CNN
@@
 P 4600 4000
 AR Path="/5F56D9CC" Ref="#PWR?"  Part="1"
-AR Path="/5F35C9AC/5F56D9CC" Ref="#PWR0131"  Part="1"
-F 0 "#PWR0131" H 4600 3750 50  0001 C CNN
+AR Path="/5F35C9AC/5F56D9CC" Ref="#PWR028"  Part="1"
+F 0 "#PWR028" H 4600 3750 50  0001 C CNN
 F 1 "GND" H 4603 3874 50  0000 C CNN
 F 2 "" H 4500 3650 50  0001 C CNN
@@
 P 4600 5050
 AR Path="/5F56D9D2" Ref="#PWR?"  Part="1"
-AR Path="/5F35C9AC/5F56D9D2" Ref="#PWR0132"  Part="1"
-F 0 "#PWR0132" H 4600 4800 50  0001 C CNN
+AR Path="/5F35C9AC/5F56D9D2" Ref="#PWR030"  Part="1"
+F 0 "#PWR030" H 4600 4800 50  0001 C CNN
 F 1 "GND" H 4603 4924 50  0000 C CNN
 F 2 "" H 4500 4700 50  0001 C CNN

Commit message: Component selection by MPN and routing cleanup
Parts:
- C23, C30, C42: MPN (none) -> CL10A106MQ8NNNC
- C24: MPN (none) -> CL10A105KB8NNNC
- C25, C26, C27, C28, C29, C31, C33, C34, C35, C36, C37, C38, C39, C40, C41, C43: MPN (none) -> CL10B104KB8NNNC
- C32: MPN (none) -> CL21A106KAYNNNE
- U1: MPN (none) -> iCE40HX4K-TQ144; manf# iCE40HX4K-TQ144 -> (none)
Changed lines of the file:
@@
 F 2 "Package_QFP:TQFP-144_20x20mm_P0.5mm" H 2000 3050 60  0001 L CNN
 F 3 "https://www.mouser.com/datasheet/2/225/FPGA-DS-02029-3-5-iCE40-LP-HX-Family-Data-Sheet-1022803.pdf" H 2000 2850 60  0001 L CNN
-F 4 "iCE40HX4K-TQ144" H 2000 2950 60  0001 L CNN "manf#"
+F 4 "" H 2000 2950 60  0001 L CNN "manf#"
+F 5 "iCE40HX4K-TQ144" H 1800 3000 50  0001 C CNN "MPN"
 	6    1800 3000
 	1    0    0    -1
@@
 F 2 "Package_QFP:TQFP-144_20x20mm_P0.5mm" H 3500 3650 60  0001 L CNN
 F 3 "https://www.mouser.com/datasheet/2/225/FPGA-DS-02029-3-5-iCE40-LP-HX-Family-Data-Sheet-1022803.pdf" H 3500 3450 60  0001 L CNN
-F 4 "iCE40HX4K-TQ144" H 3500 3550 60  0001 L CNN "manf#"
+F 4 "" H 3500 3550 60  0001 L CNN "manf#"
+F 5 "iCE40HX4K-TQ144" H 3300 3600 50  0001 C CNN "MPN"
 	7    3300 3600
 	-1   0    0    -1
@@
 F 2 "Capacitor_SMD:C_0603_1608Metric" H 5238 3500 50  0001 C CNN
 F 3 "~" H 5200 3650 50  0001 C CNN
+F 4 "CL10B104KB8NNNC" H 5200 3650 50  0001 C CNN "MPN"
 	1    5200 3650
 	1    0    0    -1
@@
 F 2 "Capacitor_SMD:C_0603_1608Metric" H 5538 3500 50  0001 C CNN
 F 3 "~" H 5500 3650 50  0001 C CNN
+F 4 "CL10B104KB8NNNC" H 5500 3650 50  0001 C CNN "MPN"
 	1    5500 3650
 	1    0    0    -1
@@
 F 2 "Capacitor_SMD:C_0603_1608Metric" H 5838 3500 50  0001 C CNN
 F 3 "~" H 5800 3650 50  0001 C CNN
+F 4 "CL10B104KB8NNNC" H 5800 3650 50  0001 C CNN "MPN"
 	1    5800 3650
 	1    0    0    -1
@@
 F 2 "Capacitor_SMD:C_0603_1608Metric" H 6138 3500 50  0001 C CNN
 F 3 "~" H 6100 3650 50  0001 C CNN
+F 4 "CL10B104KB8NNNC" H 6100 3650 50  0001 C CNN "MPN"
 	1    6100 3650
 	1    0    0    -1
@@
 F 2 "Capacitor_SMD:C_0603_1608Metric" H 8888 3500 50  0001 C CNN
 F 3 "~" H 8850 3650 50  0001 C CNN
+F 4 "CL10A106MQ8NNNC" H 8850 3650 50  0001 C CNN "MPN"
 	1    8850 3650
 	1    0    0    -1
@@
 F 2 "Capacitor_SMD:C_0603_1608Metric" H 9188 3500 50  0001 C CNN
 F 3 "~" H 9150 3650 50  0001 C CNN
+F 4 "CL10B104KB8NNNC" H 9150 3650 50  0001 C CNN "MPN"
 	1    9150 3650
 	1    0    0    -1
@@
 F 2 "Capacitor_SMD:C_0603_1608Metric" H 5538 4550 50  0001 C CNN
 F 3 "~" H 5500 4700 50  0001 C CNN
+F 4 "CL10B104KB8NNNC" H 5500 4700 50  0001 C CNN "MPN"
 	1    5500 4700
 	1    0    0    -1
@@
 F 2 "Capacitor_SMD:C_0603_1608Metric" H 5838 4550 50  0001 C CNN
 F 3 "~" H 5800 4700 50  0001 C CNN
+F 4 "CL10B104KB8NNNC" H 5800 4700 50  0001 C CNN "MPN"
 	1    5800 4700
 	1    0    0    -1
@@
 F 2 "Capacitor_SMD:C_0603_1608Metric" H 8888 4550 50  0001 C CNN
 F 3 "~" H 8850 4700 50  0001 C CNN
+F 4 "CL10A106MQ8NNNC" H 8850 4700 50  0001 C CNN "MPN"
 	1    8850 4700
 	1    0    0    -1
@@
 F 2 "Capacitor_SMD:C_0603_1608Metric" H 9188 4550 50  0001 C CNN
 F 3 "~" H 9150 4700 50  0001 C CNN
+F 4 "CL10B104KB8NNNC" H 9150 4700 50  0001 C CNN "MPN"
 	1    9150 4700
 	1    0    0    -1
@@
 F 2 "Capacitor_SMD:C_0603_1608Metric" H 4638 3500 50  0001 C CNN
 F 3 "~" H 4600 3650 50  0001 C CNN
+F 4 "CL10A106MQ8NNNC" H 4600 3650 50  0001 C CNN "MPN"
 	1    4600 3650
 	1    0    0    -1
@@
 F 2 "Capacitor_SMD:C_0603_1608Metric" H 4938 3500 50  0001 C CNN
 F 3 "~" H 4900 3650 50  0001 C CNN
+F 4 "CL10A105KB8NNNC" H 4900 3650 50  0001 C CNN "MPN"
 	1    4900 3650
 	1    0    0    -1
@@
 F 2 "Capacitor_SMD:C_0603_1608Metric" H 5238 4550 50  0001 C CNN
 F 3 "~" H 5200 4700 50  0001 C CNN
+F 4 "CL10B104KB8NNNC" H 5200 4700 50  0001 C CNN "MPN"
 	1    5200 4700
 	1    0    0    -1
@@
 F 2 "Capacitor_SMD:C_0603_1608Metric" H 4938 4550 50  0001 C CNN
 F 3 "~" H 4900 4700 50  0001 C CNN
+F 4 "CL10B104KB8NNNC" H 4900 4700 50  0001 C CNN "MPN"
 	1    4900 4700
 	1    0    0    -1
@@
 F 2 "Capacitor_SMD:C_0603_1608Metric" H 7038 4550 50  0001 C CNN
 F 3 "~" H 7000 4700 50  0001 C CNN
+F 4 "CL10B104KB8NNNC" H 7000 4700 50  0001 C CNN "MPN"
 	1    7000 4700
 	1    0    0    -1
@@
 F 2 "Capacitor_SMD:C_0603_1608Metric" H 6738 4550 50  0001 C CNN
 F 3 "~" H 6700 4700 50  0001 C CNN
+F 4 "CL10B104KB8NNNC" H 6700 4700 50  0001 C CNN "MPN"
 	1    6700 4700
 	1    0    0    -1
@@
 F 2 "Capacitor_SMD:C_0603_1608Metric" H 6438 4550 50  0001 C CNN
 F 3 "~" H 6400 4700 50  0001 C CNN
+F 4 "CL10B104KB8NNNC" H 6400 4700 50  0001 C CNN "MPN"
 	1    6400 4700
 	1    0    0    -1
@@
 F 2 "Capacitor_SMD:C_0603_1608Metric" H 6138 4550 50  0001 C CNN
 F 3 "~" H 6100 4700 50  0001 C CNN
+F 4 "CL10B104KB8NNNC" H 6100 4700 50  0001 C CNN "MPN"
 	1    6100 4700
 	1    0    0    -1
@@
 F 2 "Capacitor_SMD:C_0805_2012Metric" H 4638 4550 50  0001 C CNN
 F 3 "~" H 4600 4700 50  0001 C CNN
+F 4 "CL21A106KAYNNNE" H 4600 4700 50  0001 C CNN "MPN"
 	1    4600 4700
 	1    0    0    -1
@@
 F 2 "Capacitor_SMD:C_0603_1608Metric" H 7338 4550 50  0001 C CNN
 F 3 "~" H 7300 4700 50  0001 C CNN
+F 4 "CL10B104KB8NNNC" H 7300 4700 50  0001 C CNN "MPN"
 	1    7300 4700
 	1    0    0    -1
@@
 F 2 "Capacitor_SMD:C_0603_1608Metric" H 7338 3500 50  0001 C CNN
 F 3 "~" H 7300 3650 50  0001 C CNN
+F 4 "CL10B104KB8NNNC" H 7300 3650 50  0001 C CNN "MPN"
 	1    7300 3650
 	1    0    0    -1

Commit message: Complete component selection by MPN
Parts:
- D1: footprint Diode_SMD:D_SOD-123 -> Diode_SMD:D_SOD-123F; MPN (none) -> SBR2M60S1F-7
- R6, R7: MPN (none) -> RC0603FR-07100RL
Changed lines of the file:
@@
 F 2 "Resistor_SMD:R_0603_1608Metric" V 8530 4450 50  0001 C CNN
 F 3 "~" H 8600 4450 50  0001 C CNN
+F 4 "RC0603FR-07100RL" H 8600 4450 50  0001 C CNN "MPN"
 	1    8600 4450
 	0    1    1    0
@@
 F 2 "Resistor_SMD:R_0603_1608Metric" V 8530 3400 50  0001 C CNN
 F 3 "~" H 8600 3400 50  0001 C CNN
+F 4 "RC0603FR-07100RL" H 8600 3400 50  0001 C CNN "MPN"
 	1    8600 3400
 	0    1    1    0
@@
 F 0 "D1" H 7050 3184 50  0000 C CNN
 F 1 "~~800mVf" H 7050 3275 50  0000 C CNN
-F 2 "Diode_SMD:D_SOD-123" H 7050 3400 50  0001 C CNN
+F 2 "Diode_SMD:D_SOD-123F" H 7050 3400 50  0001 C CNN
 F 3 "~" H 7050 3400 50  0001 C CNN
+F 4 "SBR2M60S1F-7" H 7050 3400 50  0001 C CNN "MPN"
 	1    7050 3400
 	-1   0    0    1

Commit message: Rename SD_DET signal to SD_CD for consistency
Parts:
- added C45, C47: 10n, Capacitor_SMD:C_0603_1608Metric, symbol Device:C
- added C46: 1u, Capacitor_SMD:C_0603_1608Metric, symbol Device:C
- D1: symbol Device:D_Schottky -> Device:D
Connections:
- wire segments 137 -> 149
Other:
- moved on the sheet: C23, C24, C25, C26, C27, C28, C29, C30, C31, C32, C33, C34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
