File: hardware/fpga-ice40/Memory_Flash.sch (KiCad schematic (older format))
At the start: 8 parts, among them U3 W25Q32JVSS, U4 W25Q32JVSS, U5 S25FL256SAGMFI01, U6 S25FL256SAGMFI01

Commit message: Reannotate schematic symbols
Parts:
- renumbered C22 to C14, C23 to C15, U3 to U6, U6 to U7, U4 to U8
Changed lines of the file:
@@
 P 5600 5500
 AR Path="/5F8E1312" Ref="C?"  Part="1"
-AR Path="/5F8CA8A2/5F8E1312" Ref="C23"  Part="1"
-F 0 "C23" H 5550 5600 50  0000 R CNN
+AR Path="/5F8CA8A2/5F8E1312" Ref="C15"  Part="1"
+F 0 "C15" H 5550 5600 50  0000 R CNN
 F 1 "100n" H 5550 5400 50  0000 R CNN
 F 2 "Capacitor_SMD:C_0603_1608Metric" H 5638 5350 50  0001 C CNN
@@
 P 5600 3400
 AR Path="/5F8E131E" Ref="C?"  Part="1"
-AR Path="/5F8CA8A2/5F8E131E" Ref="C22"  Part="1"
-F 0 "C22" H 5550 3500 50  0000 R CNN
+AR Path="/5F8CA8A2/5F8E131E" Ref="C14"  Part="1"
+F 0 "C14" H 5550 3500 50  0000 R CNN
 F 1 "100n" H 5550 3300 50  0000 R CNN
 F 2 "Capacitor_SMD:C_0603_1608Metric" H 5638 3250 50  0001 C CNN
@@
 P 5600 5900
 AR Path="/5F8E1352" Ref="#PWR?"  Part="1"
-AR Path="/5F8CA8A2/5F8E1352" Ref="#PWR0112"  Part="1"
-F 0 "#PWR0112" H 5600 5650 50  0001 C CNN
+AR Path="/5F8CA8A2/5F8E1352" Ref="#PWR014"  Part="1"
+F 0 "#PWR014" H 5600 5650 50  0001 C CNN
 F 1 "GND" H 5603 5774 50  0000 C CNN
 F 2 "" H 5500 5550 50  0001 C CNN
@@
 P 5600 3800
 AR Path="/5F8E1358" Ref="#PWR?"  Part="1"
-AR Path="/5F8CA8A2/5F8E1358" Ref="#PWR0113"  Part="1"
-F 0 "#PWR0113" H 5600 3550 50  0001 C CNN
+AR Path="/5F8CA8A2/5F8E1358" Ref="#PWR012"  Part="1"
+F 0 "#PWR012" H 5600 3550 50  0001 C CNN
 F 1 "GND" H 5603 3674 50  0000 C CNN
 F 2 "" H 5500 3450 50  0001 C CNN
@@
 P 7900 3800
 AR Path="/5F8E1362" Ref="#PWR?"  Part="1"
-AR Path="/5F8CA8A2/5F8E1362" Ref="#PWR0114"  Part="1"
-F 0 "#PWR0114" H 7900 3550 50  0001 C CNN
+AR Path="/5F8CA8A2/5F8E1362" Ref="#PWR013"  Part="1"
+F 0 "#PWR013" H 7900 3550 50  0001 C CNN
 F 1 "GND" H 7903 3674 50  0000 C CNN
 F 2 "" H 7800 3450 50  0001 C CNN
@@
 P 7900 5900
 AR Path="/5F8E13A1" Ref="#PWR?"  Part="1"
-AR Path="/5F8CA8A2/5F8E13A1" Ref="#PWR0115"  Part="1"
-F 0 "#PWR0115" H 7900 5650 50  0001 C CNN
+AR Path="/5F8CA8A2/5F8E13A1" Ref="#PWR015"  Part="1"
+F 0 "#PWR015" H 7900 5650 50  0001 C CNN
 F 1 "GND" H 7903 5774 50  0000 C CNN
 F 2 "" H 7800 5550 50  0001 C CNN
@@
 P 7700 5000
 AR Path="/5F8E13A8" Ref="U?"  Part="1"
-AR Path="/5F8CA8A2/5F8E13A8" Ref="U6"  Part="1"
-F 0 "U6" H 8600 5150 50  0000 R CNN
+AR Path="/5F8CA8A2/5F8E13A8" Ref="U7"  Part="1"
+F 0 "U7" H 8600 5150 50  0000 R CNN
 F 1 "S25FL256SAGMFI01" H 8600 5050 50  0000 R CNN
 F 2 "Package_SO:SOIC-16W_7.5x10.3mm_P1.27mm" H 8150 4050 50  0001 C CNN
@@
 P 5400 3000
 AR Path="/5F8E13C2" Ref="U?"  Part="1"
-AR Path="/5F8CA8A2/5F8E13C2" Ref="U3"  Part="1"
-F 0 "U3" H 6300 3150 50  0000 R CNN
+AR Path="/5F8CA8A2/5F8E13C2" Ref="U6"  Part="1"
+F 0 "U6" H 6300 3150 50  0000 R CNN
 F 1 "W25Q32JVSS" H 6300 3050 50  0000 R CNN
 F 2 "local_hacks:SOIC-8_5.275x5.275mm_P1.27mm__No_CrtYd" H 5900 2150 50  0001 C CNN
@@
 P 5400 5100
 AR Path="/5F8E13C9" Ref="U?"  Part="1"
-AR Path="/5F8CA8A2/5F8E13C9" Ref="U4"  Part="1"
-F 0 "U4" H 6300 5250 50  0000 R CNN
+AR Path="/5F8CA8A2/5F8E13C9" Ref="U8"  Part="1"
+F 0 "U8" H 6300 5250 50  0000 R CNN
 F 1 "W25Q32JVSS" H 6300 5150 50  0000 R CNN
 F 2 "local_hacks:SOIC-8_5.275x5.275mm_P1.27mm__No_CrtYd" H 5900 4250 50  0001 C CNN

Commit message: Component selection by MPN and routing cleanup
Parts:
- C14, C15: MPN (none) -> CL10B104KB8NNNC
- RN1, RN2: MPN (none) -> YC164-JR-0710KL
- U5, U7: MPN (none) -> S25FL256SAGMFI01
- U6, U8: MPN (none) -> W25Q32JVSSIQ
Changed lines of the file:
@@
 F 2 "Capacitor_SMD:C_0603_1608Metric" H 5638 5350 50  0001 C CNN
 F 3 "~" H 5600 5500 50  0001 C CNN
+F 4 "CL10B104KB8NNNC" H 5600 5500 50  0001 C CNN "MPN"
 	1    5600 5500
 	-1   0    0    -1
@@
 F 2 "Capacitor_SMD:C_0603_1608Metric" H 5638 3250 50  0001 C CNN
 F 3 "~" H 5600 3400 50  0001 C CNN
+F 4 "CL10B104KB8NNNC" H 5600 3400 50  0001 C CNN "MPN"
 	1    5600 3400
 	-1   0    0    -1
@@
 F 2 "Resistor_SMD:R_Array_Convex_4x0603" V 4425 4900 50  0001 C CNN
 F 3 "~" H 4150 4900 50  0001 C CNN
+F 4 "YC164-JR-0710KL" H 4150 4900 50  0001 C CNN "MPN"
 	1    4150 4900
 	1    0    0    -1
@@
 F 2 "Package_SO:SOIC-16W_7.5x10.3mm_P1.27mm" H 8150 1950 50  0001 C CNN
 F 3 "https://www.cypress.com/file/448601/download" H 9100 2900 50  0001 C CNN
+F 4 "S25FL256SAGMFI01" H 7700 2900 50  0001 C CNN "MPN"
 	1    7700 2900
 	-1   0    0    -1
@@
 F 2 "Resistor_SMD:R_Array_Convex_4x0603" V 4425 2800 50  0001 C CNN
 F 3 "~" H 4150 2800 50  0001 C CNN
+F 4 "YC164-JR-0710KL" H 4150 2800 50  0001 C CNN "MPN"
 	1    4150 2800
 	1    0    0    -1
@@
 F 2 "Package_SO:SOIC-16W_7.5x10.3mm_P1.27mm" H 8150 4050 50  0001 C CNN
 F 3 "https://www.cypress.com/file/448601/download" H 9100 5000 50  0001 C CNN
+F 4 "S25FL256SAGMFI01" H 7700 5000 50  0001 C CNN "MPN"
 	1    7700 5000
 	-1   0    0    -1
@@
 F 2 "local_hacks:SOIC-8_5.275x5.275mm_P1.27mm__No_CrtYd" H 5900 2150 50  0001 C CNN
 F 3 "https://www.mouser.com/datasheet/2/949/w25q32jv_dtr_revg_03272018_plus-1489786.pdf" H 6400 2700 50  0001 C CNN
+F 4 "W25Q32JVSSIQ" H 5400 3000 50  0001 C CNN "MPN"
 	1    5400 3000
 	-1   0    0    -1
@@
 F 2 "local_hacks:SOIC-8_5.275x5.275mm_P1.27mm__No_CrtYd" H 5900 4250 50  0001 C CNN
 F 3 "https://www.mouser.com/datasheet/2/949/w25q32jv_dtr_revg_03272018_plus-1489786.pdf" H 6400 4800 50  0001 C CNN
+F 4 "W25Q32JVSSIQ" H 5400 5100 50  0001 C CNN "MPN"
 	1    5400 5100
 	-1   0    0    -1

Commit message: Completed verification of all pins for all symbols
Parts:
- U5, U7: value S25FL256SAGMFI01 -> S25FL256SAGMFI01x; MPN S25FL256SAGMFI01 -> S25FL256SAGMFI013
- U6, U8: value W25Q32JVSS -> W25Q32JVSSIM; MPN W25Q32JVSSIQ -> W25Q32JVSSIM (TR)
Changed lines of the file:
@@
 AR Path="/5F8CA8A2/5F8E1369" Ref="U5"  Part="1"
 F 0 "U5" H 8600 3050 50  0000 R CNN
-F 1 "S25FL256SAGMFI01" H 8600 2950 50  0000 R CNN
+F 1 "S25FL256SAGMFI01x" H 8600 2950 50  0000 R CNN
 F 2 "Package_SO:SOIC-16W_7.5x10.3mm_P1.27mm" H 8150 1950 50  0001 C CNN
 F 3 "https://www.cypress.com/file/448601/download" H 9100 2900 50  0001 C CNN
-F 4 "S25FL256SAGMFI01" H 7700 2900 50  0001 C CNN "MPN"
+F 4 "S25FL256SAGMFI013" H 7700 2900 50  0001 C CNN "MPN"
 	1    7700 2900
 	-1   0    0    -1
@@
 AR Path="/5F8CA8A2/5F8E13A8" Ref="U7"  Part="1"
 F 0 "U7" H 8600 5150 50  0000 R CNN
-F 1 "S25FL256SAGMFI01" H 8600 5050 50  0000 R CNN
+F 1 "S25FL256SAGMFI01x" H 8600 5050 50  0000 R CNN
 F 2 "Package_SO:SOIC-16W_7.5x10.3mm_P1.27mm" H 8150 4050 50  0001 C CNN
 F 3 "https://www.cypress.com/file/448601/download" H 9100 5000 50  0001 C CNN
-F 4 "S25FL256SAGMFI01" H 7700 5000 50  0001 C CNN "MPN"
+F 4 "S25FL256SAGMFI013" H 7700 5000 50  0001 C CNN "MPN"
 	1    7700 5000
 	-1   0    0    -1
@@
 AR Path="/5F8CA8A2/5F8E13C2" Ref="U6"  Part="1"
 F 0 "U6" H 6300 3150 50  0000 R CNN
-F 1 "W25Q32JVSS" H 6300 3050 50  0000 R CNN
+F 1 "W25Q32JVSSIM" H 6300 3050 50  0000 R CNN
 F 2 "local_hacks:SOIC-8_5.275x5.275mm_P1.27mm__No_CrtYd" H 5900 2150 50  0001 C CNN
 F 3 "https://www.mouser.com/datasheet/2/949/w25q32jv_dtr_revg_03272018_plus-1489786.pdf" H 6400 2700 50  0001 C CNN
-F 4 "W25Q32JVSSIQ" H 5400 3000 50  0001 C CNN "MPN"
+F 4 "W25Q32JVSSIM (TR)" H 5400 3000 50  0001 C CNN "MPN"
 	1    5400 3000
 	-1   0    0    -1
@@
 AR Path="/5F8CA8A2/5F8E13C9" Ref="U8"  Part="1"
 F 0 "U8" H 6300 5250 50  0000 R CNN
-F 1 "W25Q32JVSS" H 6300 5150 50  0000 R CNN
+F 1 "W25Q32JVSSIM" H 6300 5150 50  0000 R CNN
 F 2 "local_hacks:SOIC-8_5.275x5.275mm_P1.27mm__No_CrtYd" H 5900 4250 50  0001 C CNN
 F 3 "https://www.mouser.com/datasheet/2/949/w25q32jv_dtr_revg_03272018_plus-1489786.pdf" H 6400 4800 50  0001 C CNN
-F 4 "W25Q32JVSSIQ" H 5400 5100 50  0001 C CNN "MPN"
+F 4 "W25Q32JVSSIM (TR)" H 5400 5100 50  0001 C CNN "MPN"
 	1    5400 5100
 	-1   0    0    -1
