File: hardware/cart-ecp5/FPGA-IO.sch (KiCad schematic (older format))
At the start: 12 parts, among them J1 JTAG, U1 LFE5U-25F-xBG256x, U2 W25Q128JVPIQ, X1 XO_Generic_NC

Commit message: Check all resistor values for power management and assign MPN for caps and resistors
Parts:
- C1, C2, C45: MFR (none) -> Samsung; MPN (none) -> CL05B104KO5NNNC
- R26, R3: MFR (none) -> Yageo; MPN (none) -> RC0402FR-074K7L
- U1: MFR (none) -> Lattice
- U2: MFR (none) -> Winbond; MPN (none) -> W25Q128JVPIQ
Changed lines of the file:
@@
 F 3 "" H 6550 650 60  0001 R CNN
 F 4 "LFE5U-25F-xBG256x" H 5750 -2450 60  0001 C CNN "MPN"
+F 5 "Lattice" H 5000 1500 50  0001 C CNN "MFR"
 	2    5000 1500
 	1    0    0    -1
@@
 F 3 "" H 6550 4650 60  0001 R CNN
 F 4 "LFE5U-25F-xBG256x" H 5750 1550 60  0001 C CNN "MPN"
+F 5 "Lattice" H 5000 5500 50  0001 C CNN "MFR"
 	4    5000 5500
 	1    0    0    -1
@@
 F 3 "" H 10050 4650 60  0001 R CNN
 F 4 "LFE5U-25F-xBG256x" H 9250 1550 60  0001 C CNN "MPN"
+F 5 "Lattice" H 8500 5500 50  0001 C CNN "MFR"
 	5    8500 5500
 	1    0    0    -1
@@
 F 3 "" H 13550 4650 60  0001 R CNN
 F 4 "LFE5U-25F-xBG256x" H 12750 1550 60  0001 C CNN "MPN"
+F 5 "Lattice" H 12000 5500 50  0001 C CNN "MFR"
 	6    12000 5500
 	1    0    0    -1
@@
 F 3 "" H 10050 650 60  0001 R CNN
 F 4 "LFE5U-25F-xBG256x" H 9250 -2450 60  0001 C CNN "MPN"
+F 5 "Lattice" H 8500 1500 50  0001 C CNN "MFR"
 	7    8500 1500
 	1    0    0    -1
@@
 F 2 "Resistor_SMD:R_0402_1005Metric" V 10880 4000 50  0001 C CNN
 F 3 "~" H 10950 4000 50  0001 C CNN
+F 4 "RC0402FR-074K7L" H 10950 4000 50  0001 C CNN "MPN"
+F 5 "Yageo" H 10950 4000 50  0001 C CNN "MFR"
 	1    10950 4000
 	0    1    1    0
@@
 F 3 "" H 3050 650 60  0001 R CNN
 F 4 "LFE5U-25F-xBG256x" H 2250 -2450 60  0001 C CNN "MPN"
+F 5 "Lattice" H 1500 1500 50  0001 C CNN "MFR"
 	1    1500 1500
 	1    0    0    -1
@@
 F 3 "" H 3050 4650 60  0001 R CNN
 F 4 "LFE5U-25F-xBG256x" H 2250 1550 60  0001 C CNN "MPN"
+F 5 "Lattice" H 1500 5500 50  0001 C CNN "MFR"
 	3    1500 5500
 	1    0    0    -1
@@
 F 2 "Capacitor_SMD:C_0402_1005Metric" H 13438 1700 50  0001 C CNN
 F 3 "~" H 13400 1850 50  0001 C CNN
+F 4 "Samsung" H 13400 1850 50  0001 C CNN "MFR"
+F 5 "CL05B104KO5NNNC" H 13400 1850 50  0001 C CNN "MPN"
 	1    13400 1850
 	1    0    0    -1
@@
 F 2 "Capacitor_SMD:C_0402_1005Metric" H 13688 3100 50  0001 C CNN
 F 3 "~" H 13650 3250 50  0001 C CNN
+F 4 "Samsung" H 13650 3250 50  0001 C CNN "MFR"
+F 5 "CL05B104KO5NNNC" H 13650 3250 50  0001 C CNN "MPN"
 	1    13650 3250
 	1    0    0    -1
@@
 F 2 "Package_SON:WSON-8-1EP_6x5mm_P1.27mm_EP3.4x4mm" H 13700 650 50  0001 C CNN
 F 3 "https://www.mouser.com/datasheet/2/949/w25q128jv_revf_03272018_plus-1489608.pdf" H 14200 1200 50  0001 C CNN
+F 4 "Winbond" H 13200 1500 50  0001 C CNN "MFR"
+F 5 "W25Q128JVPIQ" H 13200 1500 50  0001 C CNN "MPN"
 	1    13200 1500
 	-1   0    0    -1
@@
 F 2 "Resistor_SMD:R_0402_1005Metric" V 10930 1950 50  0001 C CNN
 F 3 "~" H 11000 1950 50  0001 C CNN
+F 4 "RC0402FR-074K7L" H 11000 1950 50  0001 C CNN "MPN"
+F 5 "Yageo" H 11000 1950 50  0001 C CNN "MFR"
 	1    11000 1950
 	1    0    0    -1
@@
 F 2 "Capacitor_SMD:C_0402_1005Metric" H 11038 2300 50  0001 C CNN
 F 3 "~" H 11000 2450 50  0001 C CNN
+F 4 "Samsung" H 11000 2450 50  0001 C CNN "MFR"
+F 5 "CL05B104KO5NNNC" H 11000 2450 50  0001 C CNN "MPN"
 	1    11000 2450
 	1    0    0    -1
