File: hardware/cart-ecp5/FPGA-Power.sch (KiCad schematic (older format))
At the start: 18 parts, among them U1 LFE5U-25F-xBG256x

Commit message: Check all resistor values for power management and assign MPN for caps and resistors
Parts:
- C42, C44, C47, C49, C50, C51, C52, C55, C58, C59, C61: MFR (none) -> Samsung; MPN (none) -> CL05B104KO5NNNC
- C43, C46, C53, C54, C57, C62: MFR (none) -> Samsung; MPN (none) -> CL05B103KB5NNNC
- U1: MFR (none) -> Lattice
Changed lines of the file:
@@
 F 3 "" H 6750 2200 60  0001 R CNN
 F 4 "LFE5U-25F-xBG256x" H 5950 -900 60  0001 C CNN "MPN"
+F 5 "Lattice" H 5200 3050 50  0001 C CNN "MFR"
 	8    5200 3050
 	1    0    0    -1
@@
 F 3 "" H 13050 3950 60  0001 R CNN
 F 4 "LFE5U-25F-xBG256x" H 12250 850 60  0001 C CNN "MPN"
+F 5 "Lattice" H 11500 4800 50  0001 C CNN "MFR"
 	9    11500 4800
 	1    0    0    -1
@@
 F 2 "Capacitor_SMD:C_0402_1005Metric" H 4638 3250 50  0001 C CNN
 F 3 "~" H 4600 3400 50  0001 C CNN
+F 4 "Samsung" H 4600 3400 50  0001 C CNN "MFR"
+F 5 "CL05B103KB5NNNC" H 4600 3400 50  0001 C CNN "MPN"
 	1    4600 3400
 	1    0    0    -1
@@
 F 2 "Capacitor_SMD:C_0402_1005Metric" H 4338 3250 50  0001 C CNN
 F 3 "~" H 4300 3400 50  0001 C CNN
+F 4 "Samsung" H 4300 3400 50  0001 C CNN "MFR"
+F 5 "CL05B104KO5NNNC" H 4300 3400 50  0001 C CNN "MPN"
 	1    4300 3400
 	1    0    0    -1
@@
 F 2 "Capacitor_SMD:C_0402_1005Metric" H 4038 3250 50  0001 C CNN
 F 3 "~" H 4000 3400 50  0001 C CNN
+F 4 "Samsung" H 4000 3400 50  0001 C CNN "MFR"
+F 5 "CL05B103KB5NNNC" H 4000 3400 50  0001 C CNN "MPN"
 	1    4000 3400
 	1    0    0    -1
@@
 F 2 "Capacitor_SMD:C_0402_1005Metric" H 3738 3250 50  0001 C CNN
 F 3 "~" H 3700 3400 50  0001 C CNN
+F 4 "Samsung" H 3700 3400 50  0001 C CNN "MFR"
+F 5 "CL05B104KO5NNNC" H 3700 3400 50  0001 C CNN "MPN"
 	1    3700 3400
 	1    0    0    -1
@@
 F 2 "Capacitor_SMD:C_0402_1005Metric" H 4638 4150 50  0001 C CNN
 F 3 "~" H 4600 4300 50  0001 C CNN
+F 4 "Samsung" H 4600 4300 50  0001 C CNN "MFR"
+F 5 "CL05B104KO5NNNC" H 4600 4300 50  0001 C CNN "MPN"
 	1    4600 4300
 	1    0    0    -1
@@
 F 2 "Capacitor_SMD:C_0402_1005Metric" H 4338 4150 50  0001 C CNN
 F 3 "~" H 4300 4300 50  0001 C CNN
+F 4 "Samsung" H 4300 4300 50  0001 C CNN "MFR"
+F 5 "CL05B104KO5NNNC" H 4300 4300 50  0001 C CNN "MPN"
 	1    4300 4300
 	1    0    0    -1
@@
 F 2 "Capacitor_SMD:C_0402_1005Metric" H 6838 4150 50  0001 C CNN
 F 3 "~" H 6800 4300 50  0001 C CNN
+F 4 "Samsung" H 6800 4300 50  0001 C CNN "MFR"
+F 5 "CL05B104KO5NNNC" H 6800 4300 50  0001 C CNN "MPN"
 	1    6800 4300
 	1    0    0    -1
@@
 F 2 "Capacitor_SMD:C_0402_1005Metric" H 6838 3250 50  0001 C CNN
 F 3 "~" H 6800 3400 50  0001 C CNN
+F 4 "Samsung" H 6800 3400 50  0001 C CNN "MFR"
+F 5 "CL05B104KO5NNNC" H 6800 3400 50  0001 C CNN "MPN"
 	1    6800 3400
 	1    0    0    -1
@@
 F 2 "Capacitor_SMD:C_0402_1005Metric" H 6838 6850 50  0001 C CNN
 F 3 "~" H 6800 7000 50  0001 C CNN
+F 4 "Samsung" H 6800 7000 50  0001 C CNN "MFR"
+F 5 "CL05B104KO5NNNC" H 6800 7000 50  0001 C CNN "MPN"
 	1    6800 7000
 	1    0    0    -1
@@
 F 2 "Capacitor_SMD:C_0402_1005Metric" H 6838 5050 50  0001 C CNN
 F 3 "~" H 6800 5200 50  0001 C CNN
+F 4 "Samsung" H 6800 5200 50  0001 C CNN "MFR"
+F 5 "CL05B104KO5NNNC" H 6800 5200 50  0001 C CNN "MPN"
 	1    6800 5200
 	1    0    0    -1
@@
 F 2 "Capacitor_SMD:C_0402_1005Metric" H 6838 8650 50  0001 C CNN
 F 3 "~" H 6800 8800 50  0001 C CNN
+F 4 "Samsung" H 6800 8800 50  0001 C CNN "MFR"
+F 5 "CL05B104KO5NNNC" H 6800 8800 50  0001 C CNN "MPN"
 	1    6800 8800
 	1    0    0    -1
@@
 F 2 "Capacitor_SMD:C_0402_1005Metric" H 7138 5950 50  0001 C CNN
 F 3 "~" H 7100 6100 50  0001 C CNN
+F 4 "Samsung" H 7100 6100 50  0001 C CNN "MFR"
+F 5 "CL05B103KB5NNNC" H 7100 6100 50  0001 C CNN "MPN"
 	1    7100 6100
 	1    0    0    -1
@@
 F 2 "Capacitor_SMD:C_0402_1005Metric" H 6838 5950 50  0001 C CNN
 F 3 "~" H 6800 6100 50  0001 C CNN
+F 4 "Samsung" H 6800 6100 50  0001 C CNN "MFR"
+F 5 "CL05B104KO5NNNC" H 6800 6100 50  0001 C CNN "MPN"
 	1    6800 6100
 	1    0    0    -1
@@
 F 2 "Capacitor_SMD:C_0402_1005Metric" H 7138 6850 50  0001 C CNN
 F 3 "~" H 7100 7000 50  0001 C CNN
+F 4 "Samsung" H 7100 7000 50  0001 C CNN "MFR"
+F 5 "CL05B103KB5NNNC" H 7100 7000 50  0001 C CNN "MPN"
 	1    7100 7000
 	1    0    0    -1
@@
 F 2 "Capacitor_SMD:C_0402_1005Metric" H 7138 7750 50  0001 C CNN
 F 3 "~" H 7100 7900 50  0001 C CNN
+F 4 "Samsung" H 7100 7900 50  0001 C CNN "MFR"
+F 5 "CL05B103KB5NNNC" H 7100 7900 50  0001 C CNN "MPN"
 	1    7100 7900
 	1    0    0    -1
@@
 F 2 "Capacitor_SMD:C_0402_1005Metric" H 6838 7750 50  0001 C CNN
 F 3 "~" H 6800 7900 50  0001 C CNN
+F 4 "Samsung" H 6800 7900 50  0001 C CNN "MFR"
+F 5 "CL05B104KO5NNNC" H 6800 7900 50  0001 C CNN "MPN"
 	1    6800 7900
 	1    0    0    -1
@@
 F 2 "Capacitor_SMD:C_0402_1005Metric" H 7138 5050 50  0001 C CNN
 F 3 "~" H 7100 5200 50  0001 C CNN
+F 4 "Samsung" H 7100 5200 50  0001 C CNN "MFR"
+F 5 "CL05B103KB5NNNC" H 7100 5200 50  0001 C CNN "MPN"
 	1    7100 5200
 	1    0    0    -1
