File: hardware/cart-ecp5/Interface-USB.sch (KiCad schematic (older format))
At the start: 41 parts, among them J5 USB_C_USB2.0, U10 93C46BT-I_OT, U11 FT2232HQ, U3 USBLC6-2SC6, X2 DSC60xx

Commit message: Enlarge test points to 1mm diameter
Parts:
- TP14: footprint ng_test:TestPoint_Pad_D0.5mm -> TestPoint:TestPoint_Pad_D1.0mm
Changed lines of the file:
@@
 F 0 "TP14" H 10058 7218 50  0000 L CNN
 F 1 "TestPoint" H 10058 7127 50  0001 L CNN
-F 2 "ng_test:TestPoint_Pad_D0.5mm" H 10200 7100 50  0001 C CNN
+F 2 "TestPoint:TestPoint_Pad_D1.0mm" H 10200 7100 50  0001 C CNN
 F 3 "~" H 10200 7100 50  0001 C CNN
 	1    10000 7100

Commit message: Check all resistor values for power management and assign MPN for caps and resistors
Parts:
- C21, C22, C38, C5: MFR (none) -> Samsung; MPN (none) -> CL05A475KP5NRNC
- C23, C24, C26, C27, C29, C3, C30, C31, C32, C34, C36, C37, C39, C4, C40: MFR (none) -> Samsung; MPN (none) -> CL05B104KO5NNNC
- C6: MFR (none) -> Samsung; MPN (none) -> CL05B103KB5NNNC
- R1: MFR (none) -> Yageo; MPN (none) -> RC0402FR-07100KL
- R17, R18: MFR (none) -> Yageo; MPN (none) -> RC0402FR-075K1L
- R19, R21, R23, R24, R5: MFR (none) -> Yageo; MPN (none) -> RC0402FR-0710KL
- R20: MFR (none) -> Yageo; MPN (none) -> RC0402FR-072K2L
- R22: MFR (none) -> Yageo; MPN (none) -> RC0402FR-0712KL
- R3: MFR (none) -> Yageo; MPN (none) -> RC0402FR-076K8L
Changed lines of the file:
@@
 F 2 "Capacitor_SMD:C_0402_1005Metric" H 8188 6400 50  0001 C CNN
 F 3 "~" H 8150 6550 50  0001 C CNN
+F 4 "Samsung" H 8150 6550 50  0001 C CNN "MFR"
+F 5 "CL05B104KO5NNNC" H 8150 6550 50  0001 C CNN "MPN"
 	1    8150 6550
 	1    0    0    -1
@@
 F 2 "Resistor_SMD:R_0402_1005Metric" V 9380 5950 50  0001 C CNN
 F 3 "~" H 9450 5950 50  0001 C CNN
+F 4 "RC0402FR-0710KL" H 9450 5950 50  0001 C CNN "MPN"
+F 5 "Yageo" H 9450 5950 50  0001 C CNN "MFR"
 	1    9450 5950
 	1    0    0    -1
@@
 F 2 "Resistor_SMD:R_0402_1005Metric" V 9480 5950 50  0001 C CNN
 F 3 "~" H 9550 5950 50  0001 C CNN
+F 4 "RC0402FR-0710KL" H 9550 5950 50  0001 C CNN "MPN"
+F 5 "Yageo" H 9550 5950 50  0001 C CNN "MFR"
 	1    9550 5950
 	1    0    0    -1
@@
 F 2 "Capacitor_SMD:C_0402_1005Metric" H 8738 7300 50  0001 C CNN
 F 3 "~" H 8700 7450 50  0001 C CNN
+F 4 "Samsung" H 8700 7450 50  0001 C CNN "MFR"
+F 5 "CL05B104KO5NNNC" H 8700 7450 50  0001 C CNN "MPN"
 	1    8700 7450
 	1    0    0    -1
@@
 F 2 "Capacitor_SMD:C_0402_1005Metric" H 10088 4000 50  0001 C CNN
 F 3 "~" H 10050 4150 50  0001 C CNN
+F 4 "Samsung" H 10050 4150 50  0001 C CNN "MFR"
+F 5 "CL05A475KP5NRNC" H 10050 4150 50  0001 C CNN "MPN"
 	1    10050 4150
 	-1   0    0    -1
@@
 F 2 "Capacitor_SMD:C_0402_1005Metric" H 10388 4000 50  0001 C CNN
 F 3 "~" H 10350 4150 50  0001 C CNN
+F 4 "Samsung" H 10350 4150 50  0001 C CNN "MFR"
+F 5 "CL05B104KO5NNNC" H 10350 4150 50  0001 C CNN "MPN"
 	1    10350 4150
 	-1   0    0    -1
@@
 F 2 "Capacitor_SMD:C_0402_1005Metric" H 4438 6600 50  0001 C CNN
 F 3 "~" H 4400 6750 50  0001 C CNN
+F 4 "Samsung" H 4400 6750 50  0001 C CNN "MFR"
+F 5 "CL05A475KP5NRNC" H 4400 6750 50  0001 C CNN "MPN"
 	1    4400 6750
 	1    0    0    -1
@@
 F 2 "Capacitor_SMD:C_0402_1005Metric" H 4738 6600 50  0001 C CNN
 F 3 "~" H 4700 6750 50  0001 C CNN
+F 4 "Samsung" H 4700 6750 50  0001 C CNN "MFR"
+F 5 "CL05B104KO5NNNC" H 4700 6750 50  0001 C CNN "MPN"
 	1    4700 6750
 	1    0    0    -1
@@
 F 2 "Resistor_SMD:R_0402_1005Metric" V 10130 6600 50  0001 C CNN
 F 3 "~" H 10200 6600 50  0001 C CNN
+F 4 "RC0402FR-072K2L" H 10200 6600 50  0001 C CNN "MPN"
+F 5 "Yageo" H 10200 6600 50  0001 C CNN "MFR"
 	1    10200 6600
 	0    1    1    0
@@
 F 2 "Capacitor_SMD:C_0402_1005Metric" H 6488 3000 50  0001 C CNN
 F 3 "~" H 6450 3150 50  0001 C CNN
-F 4 "" H 6450 3150 50  0001 C CNN "MPN"
+F 4 "CL05B104KO5NNNC" H 6450 3150 50  0001 C CNN "MPN"
+F 5 "Samsung" H 6450 3150 50  0001 C CNN "MFR"
 	1    6450 3150
 	1    0    0    -1
@@
 F 2 "Resistor_SMD:R_0402_1005Metric" V 3780 5150 50  0001 C CNN
 F 3 "~" H 3850 5150 50  0001 C CNN
-F 4 "" H 3850 5150 50  0001 C CNN "MPN"
+F 4 "RC0402FR-07100KL" H 3850 5150 50  0001 C CNN "MPN"
+F 5 "Yageo" H 3850 5150 50  0001 C CNN "MFR"
 	1    3850 5150
 	1    0    0    -1
@@
 F 2 "Capacitor_SMD:C_0402_1005Metric" H 3588 5000 50  0001 C CNN
 F 3 "~" H 3550 5150 50  0001 C CNN
-F 4 "" H 3550 5150 50  0001 C CNN "MPN"
+F 4 "CL05B103KB5NNNC" H 3550 5150 50  0001 C CNN "MPN"
+F 5 "Samsung" H 3550 5150 50  0001 C CNN "MFR"
 	1    3550 5150
 	1    0    0    -1
@@
 F 2 "Capacitor_SMD:C_0402_1005Metric" H 6788 3000 50  0001 C CNN
 F 3 "~" H 6750 3150 50  0001 C CNN
-F 4 "" H 6750 3150 50  0001 C CNN "MPN"
+F 4 "CL05A475KP5NRNC" H 6750 3150 50  0001 C CNN "MPN"
+F 5 "Samsung" H 6750 3150 50  0001 C CNN "MFR"
 	1    6750 3150
 	1    0    0    -1
@@
 F 2 "Capacitor_SMD:C_0402_1005Metric" H 5988 3000 50  0001 C CNN
 F 3 "~" H 5950 3150 50  0001 C CNN
-F 4 "" H 5950 3150 50  0001 C CNN "MPN"
+F 4 "CL05B104KO5NNNC" H 5950 3150 50  0001 C CNN "MPN"
+F 5 "Samsung" H 5950 3150 50  0001 C CNN "MFR"
 	1    5950 3150
 	1    0    0    -1
@@
 F 2 "Capacitor_SMD:C_0402_1005Metric" H 4438 7650 50  0001 C CNN
 F 3 "~" H 4400 7800 50  0001 C CNN
+F 4 "Samsung" H 4400 7800 50  0001 C CNN "MFR"
+F 5 "CL05A475KP5NRNC" H 4400 7800 50  0001 C CNN "MPN"
 	1    4400 7800
 	1    0    0    -1
@@
 F 2 "Capacitor_SMD:C_0402_1005Metric" H 4738 7650 50  0001 C CNN
 F 3 "~" H 4700 7800 50  0001 C CNN
+F 4 "Samsung" H 4700 7800 50  0001 C CNN "MFR"
+F 5 "CL05B104KO5NNNC" H 4700 7800 50  0001 C CNN "MPN"
 	1    4700 7800
 	1    0    0    -1
@@
 F 2 "Capacitor_SMD:C_0402_1005Metric" H 5838 6600 50  0001 C CNN
 F 3 "~" H 5800 6750 50  0001 C CNN
+F 4 "Samsung" H 5800 6750 50  0001 C CNN "MFR"
+F 5 "CL05B104KO5NNNC" H 5800 6750 50  0001 C CNN "MPN"
 	1    5800 6750
 	1    0    0    -1
@@
 F 2 "Capacitor_SMD:C_0402_1005Metric" H 6138 6600 50  0001 C CNN
 F 3 "~" H 6100 6750 50  0001 C CNN
+F 4 "Samsung" H 6100 6750 50  0001 C CNN "MFR"
+F 5 "CL05B104KO5NNNC" H 6100 6750 50  0001 C CNN "MPN"
 	1    6100 6750
 	1    0    0    -1
@@
 F 2 "Capacitor_SMD:C_0402_1005Metric" H 6438 6600 50  0001 C CNN
 F 3 "~" H 6400 6750 50  0001 C CNN
+F 4 "Samsung" H 6400 6750 50  0001 C CNN "MFR"
+F 5 "CL05B104KO5NNNC" H 6400 6750 50  0001 C CNN "MPN"
 	1    6400 6750
 	1    0    0    -1
@@
 F 2 "Capacitor_SMD:C_0402_1005Metric" H 6738 7650 50  0001 C CNN
 F 3 "~" H 6700 7800 50  0001 C CNN
+F 4 "Samsung" H 6700 7800 50  0001 C CNN "MFR"
+F 5 "CL05B104KO5NNNC" H 6700 7800 50  0001 C CNN "MPN"
 	1    6700 7800
 	1    0    0    -1
@@
 F 2 "Capacitor_SMD:C_0402_1005Metric" H 6438 7650 50  0001 C CNN
 F 3 "~" H 6400 7800 50  0001 C CNN
+F 4 "Samsung" H 6400 7800 50  0001 C CNN "MFR"
+F 5 "CL05B104KO5NNNC" H 6400 7800 50  0001 C CNN "MPN"
 	1    6400 7800
 	1    0    0    -1
@@
 F 2 "Capacitor_SMD:C_0402_1005Metric" H 6138 7650 50  0001 C CNN
 F 3 "~" H 6100 7800 50  0001 C CNN
+F 4 "Samsung" H 6100 7800 50  0001 C CNN "MFR"
+F 5 "CL05B104KO5NNNC" H 6100 7800 50  0001 C CNN "MPN"
 	1    6100 7800
 	1    0    0    -1
@@
 F 2 "Capacitor_SMD:C_0402_1005Metric" H 5838 7650 50  0001 C CNN
 F 3 "~" H 5800 7800 50  0001 C CNN
+F 4 "Samsung" H 5800 7800 50  0001 C CNN "MFR"
+F 5 "CL05B104KO5NNNC" H 5800 7800 50  0001 C CNN "MPN"
 	1    5800 7800
 	1    0    0    -1
@@
 F 2 "Resistor_SMD:R_0402_1005Metric" V 9280 5950 50  0001 C CNN
 F 3 "~" H 9350 5950 50  0001 C CNN
-F 4 "" V 9350 5950 50  0001 C CNN "MPN"
+F 4 "RC0402FR-0710KL" V 9350 5950 50  0001 C CNN "MPN"
+F 5 "Yageo" H 9350 5950 50  0001 C CNN "MFR"
 	1    9350 5950
 	1    0    0    -1
@@
 F 2 "Resistor_SMD:R_0402_1005Metric" V 10230 5800 50  0001 C CNN
 F 3 "~" H 10300 5800 50  0001 C CNN
+F 4 "RC0402FR-0712KL" H 10300 5800 50  0001 C CNN "MPN"
+F 5 "Yageo" H 10300 5800 50  0001 C CNN "MFR"
 	1    10300 5800
 	0    1    1    0
@@
 F 2 "Resistor_SMD:R_0402_1005Metric" V 10230 5600 50  0001 C CNN
 F 3 "~" H 10300 5600 50  0001 C CNN
+F 4 "RC0402FR-0710KL" H 10300 5600 50  0001 C CNN "MPN"
+F 5 "Yageo" H 10300 5600 50  0001 C CNN "MFR"
 	1    10300 5600
 	0    1    1    0
@@
 F 2 "Resistor_SMD:R_0402_1005Metric" V 5180 3450 50  0001 C CNN
 F 3 "~" H 5250 3450 50  0001 C CNN
+F 4 "RC0402FR-075K1L" H 5250 3450 50  0001 C CNN "MPN"
+F 5 "Yageo" H 5250 3450 50  0001 C CNN "MFR"
 	1    5250 3450
 	1    0    0    -1
@@
 F 2 "Resistor_SMD:R_0402_1005Metric" V 5480 3450 50  0001 C CNN
 F 3 "~" H 5550 3450 50  0001 C CNN
+F 4 "RC0402FR-075K1L" H 5550 3450 50  0001 C CNN "MPN"
+F 5 "Yageo" H 5550 3450 50  0001 C CNN "MFR"
 	1    5550 3450
 	1    0    0    -1
@@
 F 2 "Resistor_SMD:R_0402_1005Metric" V 6380 4700 50  0001 C CNN
 F 3 "~" H 6450 4700 50  0001 C CNN
-F 4 "" H 6450 4700 50  0001 C CNN "MPN"
+F 4 "RC0402FR-076K8L" H 6450 4700 50  0001 C CNN "MPN"
+F 5 "Yageo" H 6450 4700 50  0001 C CNN "MFR"
 	1    6450 4700
 	1    0    0    -1
@@
 F 2 "Resistor_SMD:R_0402_1005Metric" V 6380 5200 50  0001 C CNN
 F 3 "~" H 6450 5200 50  0001 C CNN
-F 4 "" H 6450 5200 50  0001 C CNN "MPN"
+F 4 "RC0402FR-0710KL" H 6450 5200 50  0001 C CNN "MPN"
+F 5 "Yageo" H 6450 5200 50  0001 C CNN "MFR"
 	1    6450 5200
 	1    0    0    -1
@@
 F 2 "Capacitor_SMD:C_0402_1005Metric" H 9488 4000 50  0001 C CNN
 F 3 "~" H 9450 4150 50  0001 C CNN
+F 4 "Samsung" H 9450 4150 50  0001 C CNN "MFR"
+F 5 "CL05B104KO5NNNC" H 9450 4150 50  0001 C CNN "MPN"
 	1    9450 4150
 	-1   0    0    -1

Commit message: Update project to KiCad 5.1.9
Parts:
- J5: symbol Connector:USB_C_Receptacle_USB2.0 -> cart-ecp5-rescue:USB_C_Receptacle_USB2.0-Connector
Changed lines of the file:
@@
 $EndComp
 $Comp
-L Connector:USB_C_Receptacle_USB2.0 J5
+L cart-ecp5-rescue:USB_C_Receptacle_USB2.0-Connector J5
 U 1 1 5F216B5E
 P 3850 3500

Commit message: Reassign symbols that were rescued during update
Parts:
- J5: symbol cart-ecp5-rescue:USB_C_Receptacle_USB2.0-Connector -> Connector:USB_C_Receptacle_USB2.0
Changed lines of the file:
@@
 $EndComp
 $Comp
-L cart-ecp5-rescue:USB_C_Receptacle_USB2.0-Connector J5
+L Connector:USB_C_Receptacle_USB2.0 J5
 U 1 1 5F216B5E
 P 3850 3500

Commit message: Assign MPN for all other components except oscillators
Parts:
- FB1: MFR (none) -> TDK; MPN (none) -> MPZ1005S330HT000
- FB2, FB3: MFR (none) -> Murata; MPN (none) -> BLM15PX601SN1D
- J5: MFR (none) -> HRO; MPN (none) -> TYPE-C-31-M-12
- U10: MFR (none) -> Microchip; MPN (none) -> 93C46BT-I/OT
- U11: MFR (none) -> FTDI; MPN (none) -> FT2232HQ
- U3: MFR (none) -> ST; MPN (none) -> USBLC6-2SC6
Changed lines of the file:
@@
 F 2 "Package_TO_SOT_SMD:SOT-23-6" H 8850 6250 50  0001 C CNN
 F 3 "http://ww1.microchip.com/downloads/en/DeviceDoc/20001749K.pdf" H 8850 6500 50  0001 C CNN
+F 4 "Microchip" H 8850 6500 50  0001 C CNN "MFR"
+F 5 "93C46BT-I/OT" H 8850 6500 50  0001 C CNN "MPN"
 	1    8850 6500
 	1    0    0    -1
@@
 F 2 "Package_TO_SOT_SMD:SOT-23-6" H 4400 5400 50  0001 C CNN
 F 3 "http://www2.st.com/resource/en/datasheet/CD00050750.pdf" H 5350 5350 50  0001 C CNN
+F 4 "ST" H 5150 5000 50  0001 C CNN "MFR"
+F 5 "USBLC6-2SC6" H 5150 5000 50  0001 C CNN "MPN"
 	1    5150 5000
 	1    0    0    -1
@@
 F 2 "Inductor_SMD:L_0402_1005Metric" V 6130 2900 50  0001 C CNN
 F 3 "~" H 6200 2900 50  0001 C CNN
+F 4 "TDK" H 6200 2900 50  0001 C CNN "MFR"
+F 5 "MPZ1005S330HT000" H 6200 2900 50  0001 C CNN "MPN"
 	1    6200 2900
 	0    1    1    0
@@
 F 2 "Inductor_SMD:L_0402_1005Metric" V 4080 6500 50  0001 C CNN
 F 3 "~" H 4150 6500 50  0001 C CNN
-F 4 "" V 4150 6500 50  0001 C CNN "MPN"
+F 4 "BLM15PX601SN1D" V 4150 6500 50  0001 C CNN "MPN"
+F 5 "Murata" H 4150 6500 50  0001 C CNN "MFR"
 	1    4150 6500
 	0    1    1    0
@@
 F 2 "Inductor_SMD:L_0402_1005Metric" V 4080 7550 50  0001 C CNN
 F 3 "~" H 4150 7550 50  0001 C CNN
-F 4 "" V 4150 7550 50  0001 C CNN "MPN"
+F 4 "BLM15PX601SN1D" V 4150 7550 50  0001 C CNN "MPN"
+F 5 "Murata" H 4150 7550 50  0001 C CNN "MFR"
 	1    4150 7550
 	0    1    1    0
@@
 F 2 "ng_conn:USB_C_Receptacle_HRO_TYPE-C-31-M-12" H 4000 3500 50  0001 C CNN
 F 3 "https://www.usb.org/sites/default/files/documents/usb_type-c.zip" H 4000 3500 50  0001 C CNN
+F 4 "HRO" H 3850 3500 50  0001 C CNN "MFR"
+F 5 "TYPE-C-31-M-12" H 3850 3500 50  0001 C CNN "MPN"
 	1    3850 3500
 	1    0    0    -1
@@
 F 2 "Package_DFN_QFN:QFN-64-1EP_9x9mm_P0.5mm_EP4.35x4.35mm" H 11750 5600 50  0001 C CNN
 F 3 "https://www.ftdichip.com/Support/Documents/DataSheets/ICs/DS_FT2232H.pdf" H 11750 5600 50  0001 C CNN
+F 4 "FTDI" H 11750 5600 50  0001 C CNN "MFR"
+F 5 "FT2232HQ" H 11750 5600 50  0001 C CNN "MPN"
 	1    11750 5600
 	1    0    0    -1

Commit message: Replace 2.5x2.0mm oscillators with SiT2001B SOT23-5 oscillators
Parts:
- removed X2: DSC60xx, ng_time:Oscillator_2.5x2.0, symbol ng_osc:DSC60xx
- added R29: 10k, Resistor_SMD:R_0402_1005Metric, symbol Device:R
- added X2: SiT2001B, Package_TO_SOT_SMD:SOT-23-5, symbol ng_osc:SiT2001B
Connections:
- net GND: now also X2.1 (GND)
- net P3V3: now also R29.1, X2.4 (VDD)
- net USB_CLK: now also X2.5 (OUT)
- new net: R29.2, X2.3 (OE/~ST~/NC)
Other:
- moved on the sheet: C37
Changed lines of the file:
@@
-	1    0    0    -1
-$EndComp
-$Comp
-L ng_osc:DSC60xx X2
-U 1 1 5F1F4760
-P 9450 7300
-F 0 "X2" H 9100 7650 50  0000 L CNN
-F 1 "DSC60xx" H 9100 7550 50  0000 L CNN
-F 2 "ng_time:Oscillator_2.5x2.0" H 10150 6950 50  0001 C CNN
-F 3 "" H 9350 7300 50  0001 C CNN
-F 4 "12 MHz" H 9800 7550 50  0000 R CNN "Freq"
-	1    9450 7300
 	1    0    0    -1
 $EndComp
@@
 L Device:C C37
 U 1 1 5F1F476F
-P 8700 7450
-F 0 "C37" H 8500 7550 50  0000 L CNN
-F 1 "100n" H 8450 7350 50  0000 L CNN
-F 2 "Capacitor_SMD:C_0402_1005Metric" H 8738 7300 50  0001 C CNN
-F 3 "~" H 8700 7450 50  0001 C CNN
-F 4 "Samsung" H 8700 7450 50  0001 C CNN "MFR"
-F 5 "CL05B104KO5NNNC" H 8700 7450 50  0001 C CNN "MPN"
-	1    8700 7450
-	1    0    0    -1
-$EndComp
-Wire Wire Line
-	8700 7600 8700 7700
-Wire Wire Line
-	9000 7400 8900 7400
-Wire Wire Line
-	8900 7400 8900 7200
-Wire Wire Line
-	8900 7200 9000 7200
+P 8300 7450
+F 0 "C37" H 8100 7550 50  0000 L CNN
+F 1 "100n" H 8050 7350 50  0000 L CNN
+F 2 "Capacitor_SMD:C_0402_1005Metric" H 8338 7300 50  0001 C CNN
+F 3 "~" H 8300 7450 50  0001 C CNN
+F 4 "Samsung" H 8300 7450 50  0001 C CNN "MFR"
+F 5 "CL05B104KO5NNNC" H 8300 7450 50  0001 C CNN "MPN"
+	1    8300 7450
+	1    0    0    -1
+$EndComp
+Wire Wire Line
+	8300 7600 8300 7700
+Wire Wire Line
+	8600 7400 8500 7400
+Wire Wire Line
+	8500 7400 8500 7200
+Wire Wire Line
+	8500 7200 9000 7200
 Wire Wire Line
 	10050 4400 10350 4400
@@
 	8150 6300 8150 6400
 Wire Wire Line
-	8900 7200 8700 7200
-Connection ~ 8900 7200
-Wire Wire Line
-	8700 7200 8700 7300
+	8500 7200 8300 7200
+Connection ~ 8500 7200
+Wire Wire Line
+	8300 7200 8300 7300
 $Comp
 L Device:C C21
@@
 L ng_power:GND #PWR0116
 U 1 1 5F44F69A
-P 8700 7700
+P 8300 7700
 AR Path="/5F44F69A" Ref="#PWR0116"  Part="1"
 AR Path="/5F302051/5F44F69A" Ref="#PWR?"  Part="1"
 AR Path="/5F4552C5/5F44F69A" Ref="#PWR043"  Part="1"
-F 0 "#PWR043" H 8700 7450 50  0001 C CNN
-F 1 "GND" H 8703 7574 50  0000 C CNN
-F 2 "" H 8600 7350 50  0001 C CNN
-F 3 "" H 8700 7700 50  0001 C CNN
-	1    8700 7700
+F 0 "#PWR043" H 8300 7450 50  0001 C CNN
+F 1 "GND" H 8303 7574 50  0000 C CNN
+F 2 "" H 8200 7350 50  0001 C CNN
+F 3 "" H 8300 7700 50  0001 C CNN
+	1    8300 7700
 	1    0    0    -1
 $EndComp
@@
 P3V3
 Wire Wire Line
-	8700 7200 8600 7200
-Text GLabel 8600 7200 0    50   UnSpc ~ 0
+	8300 7200 8200 7200
+Text GLabel 8200 7200 0    50   UnSpc ~ 0
 P3V3
 Text GLabel 10050 5600 0    50   UnSpc ~ 0
@@
 Text GLabel 11950 3200 1    50   UnSpc ~ 0
 P3V3
-Connection ~ 8700 7200
+Connection ~ 8300 7200
 Connection ~ 5800 6500
 Connection ~ 5800 7550
@@
 Wire Wire Line
 	10000 7200 10550 7200
+$Comp
+L ng_osc:SiT2001B X2
+U 1 1 601D27EA
+P 9450 7300
+F 0 "X2" H 9100 7650 50  0000 L CNN
+F 1 "SiT2001B" H 9100 7550 50  0000 L CNN
+F 2 "Package_TO_SOT_SMD:SOT-23-5" H 9450 7000 50  0001 C CNN
+F 3 "https://www.mouser.com/datasheet/2/371/SiT2001B-datasheet_0-1369642.pdf" H 9400 7300 50  0001 C CNN
+F 4 "12 MHz" H 9800 7550 50  0000 R CNN "Frequency"
+F 5 "SiTime" H 9450 7300 50  0001 C CNN "MFR"
+F 6 "SiT2001BI-S2-33E-12.000000G" H 9450 7300 50  0001 C CNN "MPN"
+	1    9450 7300
+	1    0    0    -1
+$EndComp
+$Comp
+L Device:R R29
+U 1 1 601D37EA
+P 8750 7400
+F 0 "R29" V 8650 7400 50  0000 C CNN
+F 1 "10k" V 8550 7400 50  0000 C CNN
+F 2 "Resistor_SMD:R_0402_1005Metric" V 8680 7400 50  0001 C CNN
+F 3 "~" H 8750 7400 50  0001 C CNN
+F 4 "Yageo" H 8750 7400 50  0001 C CNN "MFR"
+F 5 "RC0402FR-0710KL" H 8750 7400 50  0001 C CNN "MPN"
+	1    8750 7400
+	0    -1   -1   0
+$EndComp
+Wire Wire Line
+	8900 7400 9000 7400
 $EndSCHEMATC
