File: hardware/cart-ecp5/Interface-N64.sch (KiCad schematic (older format))
At the start: 11 parts, among them J3 N64_Cartridge_Bus, U4 ATtiny25-20SU

Commit message: Assign MPN for all other components except oscillators
Parts:
- U4: value ATtiny25-20SU -> ATtiny45-20SU; MFR (none) -> Microchip; MPN (none) -> ATTINY45-20SU
Changed lines of the file:
@@
 P 8100 4950
 F 0 "U4" H 7550 4850 50  0000 R CNN
-F 1 "ATtiny25-20SU" H 7550 4750 50  0000 R CNN
+F 1 "ATtiny45-20SU" H 7550 4750 50  0000 R CNN
 F 2 "Package_SO:SOIJ-8_5.3x5.3mm_P1.27mm" H 8100 4950 50  0001 C CIN
 F 3 "http://ww1.microchip.com/downloads/en/DeviceDoc/atmel-2586-avr-8-bit-microcontroller-attiny25-attiny45-attiny85_datasheet.pdf" H 8100 4950 50  0001 C CNN
+F 4 "Microchip" H 8100 4950 50  0001 C CNN "MFR"
+F 5 "ATTINY45-20SU" H 8100 4950 50  0001 C CNN "MPN"
 	1    8100 4950
 	-1   0    0    -1

Commit message: Fix for ATtiny45 MPN
Parts:
- U4: value ATtiny45-20SU -> ATtiny45-20SUR; MPN ATTINY45-20SU -> ATTINY45-20SUR
Changed lines of the file:
@@
 P 8100 4950
 F 0 "U4" H 7550 4850 50  0000 R CNN
-F 1 "ATtiny45-20SU" H 7550 4750 50  0000 R CNN
+F 1 "ATtiny45-20SUR" H 7550 4750 50  0000 R CNN
 F 2 "Package_SO:SOIJ-8_5.3x5.3mm_P1.27mm" H 8100 4950 50  0001 C CIN
 F 3 "http://ww1.microchip.com/downloads/en/DeviceDoc/atmel-2586-avr-8-bit-microcontroller-attiny25-attiny45-attiny85_datasheet.pdf" H 8100 4950 50  0001 C CNN
 F 4 "Microchip" H 8100 4950 50  0001 C CNN "MFR"
-F 5 "ATTINY45-20SU" H 8100 4950 50  0001 C CNN "MPN"
+F 5 "ATTINY45-20SUR" H 8100 4950 50  0001 C CNN "MPN"
 	1    8100 4950
 	-1   0    0    -1
