File: hardware/cart-ecp5/Power.kicad_sch (KiCad schematic)
At the start: 49 parts, among them J4 Conn_01x02, U13 TLV62568DBV, U5 TPS2111A, U6 TLV62568DBV, U7 TLV62568DBV, U8 TLV73325PDBV

Commit message: hardware: Substitute library symbol for USB-C connector
Parts:
- renumbered C3 to C5, C52 to C6, C4 to C7, C53 to C8, C51 to C9
Changed lines of the file:
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@@
 	(label "FB_1V1"
 		(at 201.93 87.63 0)
+		(fields_autoplaced yes)
 		(effects
 			(font
@@
 	(label "SW_1V8"
 		(at 201.93 128.27 0)
+		(fields_autoplaced yes)
 		(effects
 			(font
@@
 	(label "FB_3V3"
 		(at 201.93 41.91 0)
+		(fields_autoplaced yes)
 		(effects
 			(font
@@
 	(label "SW_1V1"
 		(at 201.93 82.55 0)
+		(fields_autoplaced yes)
 		(effects
 			(font
@@
 	(label "SW_3V3"
 		(at 201.93 36.83 0)
+		(fields_autoplaced yes)
 		(effects
 			(font
@@
 	(label "FB_1V8"
 		(at 201.93 133.35 0)
+		(fields_autoplaced yes)
 		(effects
 			(font
@@
 		(on_board yes)
 		(dnp no)
-		(property "Reference" "C53"
+		(property "Reference" "C8"
 			(at 76.2 43.18 0)
 			(effects
@@
 		(instances
 			(project "cart-ecp5"
-				(path "/d0de5b81-cadf-4377-8c13-b4d382700369"
-					(reference "C?")
-					(unit 1)
-				)
 				(path "/d0de5b81-cadf-4377-8c13-b4d382700369/00000000-0000-0000-0000-00005f483803"
 					(reference "C8")
@@
 		(on_board yes)
 		(dnp no)
-		(property "Reference" "C52"
+		(property "Reference" "C6"
 			(at 60.96 43.18 0)
 			(effects
@@
 		(instances
 			(project "cart-ecp5"
-				(path "/d0de5b81-cadf-4377-8c13-b4d382700369"
-					(reference "C?")
-					(unit 1)
-				)
 				(path "/d0de5b81-cadf-4377-8c13-b4d382700369/00000000-0000-0000-0000-00005f483803"
 					(reference "C6")
@@
 		(on_board yes)
 		(dnp no)
-		(property "Reference" "C51"
+		(property "Reference" "C9"
 			(at 127 40.64 0)
 			(effects
@@
 		(instances
 			(project "cart-ecp5"
-				(path "/d0de5b81-cadf-4377-8c13-b4d382700369"
-					(reference "C?")
-					(unit 1)
-				)
 				(path "/d0de5b81-cadf-4377-8c13-b4d382700369/00000000-0000-0000-0000-00005f483803"
 					(reference "C9")
@@
 		(instances
 			(project "cart-ecp5"
-				(path "/d0de5b81-cadf-4377-8c13-b4d382700369"
-					(reference "#PWR?")
-					(unit 1)
-				)
 				(path "/d0de5b81-cadf-4377-8c13-b4d382700369/00000000-0000-0000-0000-00005f483803"
 					(reference "#PWR0101")
@@
 		(on_board yes)
 		(dnp no)
-		(property "Reference" "C4"
+		(property "Reference" "C7"
 			(at 68.58 43.18 0)
 			(effects
@@
 		(instances
 			(project "cart-ecp5"
-				(path "/d0de5b81-cadf-4377-8c13-b4d382700369"
-					(reference "C?")
-					(unit 1)
-				)
 				(path "/d0de5b81-cadf-4377-8c13-b4d382700369/00000000-0000-0000-0000-00005f483803"
 					(reference "C7")
@@
 		(on_board yes)
 		(dnp no)
-		(property "Reference" "C3"
+		(property "Reference" "C5"
 			(at 53.34 43.18 0)
 			(effects
@@
 		(instances
 			(project "cart-ecp5"
-				(path "/d0de5b81-cadf-4377-8c13-b4d382700369"
-					(reference "C?")
-					(unit 1)
-				)
 				(path "/d0de5b81-cadf-4377-8c13-b4d382700369/00000000-0000-0000-0000-00005f483803"
 					(reference "C5")
