File: hardware/cart-ecp5/FPGA-IO.kicad_sch (KiCad schematic)
At the start: 14 parts, among them J1 JTAG, U1 LFE5U-25F-xBG256x, U2 W25Q128JVPIQ, X1 SiT2001B

Commit message: hardware: Use Tag-Connect for JTAG interface
Parts:
- J1: footprint ng_conn:Samtec_FTSH-105-XX-X-DV-Mating -> Connector:Tag-Connect_TC2050-IDC-FP_2x05_P1.27mm_Vertical
Changed lines of the file:
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@@
 			)
 		)
-		(property "Footprint" "ng_conn:Samtec_FTSH-105-XX-X-DV-Mating"
+		(property "Footprint" "Connector:Tag-Connect_TC2050-IDC-FP_2x05_P1.27mm_Vertical"
 			(at 321.31 106.68 0)
 			(effects
