File: hardware/cart-ecp5/Interface-N64.kicad_sch (KiCad schematic)
At the start: 11 parts, among them J3 N64_Cartridge_Bus, U4 ATtiny45-20SUR

Commit message: hardware: Substitute library symbol for USB-C connector
Parts:
- gave numbers to parts that had none: 1
- renumbered RN4 to RN1, RN6 to RN2, RN8 to RN3, RN5 to RN4, RN7 to RN5, RN9 to RN6
Changed lines of the file:
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@@
 	(label "xN64_ALE_L"
 		(at 170.18 74.93 180)
+		(fields_autoplaced yes)
 		(effects
 			(font
@@
 	(label "xN64_AD3"
 		(at 170.18 52.07 180)
+		(fields_autoplaced yes)
 		(effects
 			(font
@@
 	(label "xN64_AD12"
 		(at 100.33 92.71 0)
+		(fields_autoplaced yes)
 		(effects
 			(font
@@
 	(label "xN64_AD6"
 		(at 217.17 57.15 180)
+		(fields_autoplaced yes)
 		(effects
 			(font
@@
 	(label "xN64_AD10"
 		(at 100.33 87.63 0)
+		(fields_autoplaced yes)
 		(effects
 			(font
@@
 	(label "xN64_CIC_DATA1"
 		(at 217.17 85.09 180)
+		(fields_autoplaced yes)
 		(effects
 			(font
@@
 	(label "xN64_AD2"
 		(at 100.33 67.31 0)
+		(fields_autoplaced yes)
 		(effects
 			(font
@@
 	(label "xN64_AD1"
 		(at 100.33 64.77 0)
+		(fields_autoplaced yes)
 		(effects
 			(font
@@
 	(label "xN64_AD8"
 		(at 217.17 49.53 180)
+		(fields_autoplaced yes)
 		(effects
 			(font
@@
 	(label "xN64_COLD_RESET#"
 		(at 217.17 69.85 180)
+		(fields_autoplaced yes)
 		(effects
 			(font
@@
 	(label "xN64_COLD_RESET#"
 		(at 100.33 125.73 0)
+		(fields_autoplaced yes)
 		(effects
 			(font
@@
 	(label "xN64_OS_EVENT#"
 		(at 100.33 128.27 0)
+		(fields_autoplaced yes)
 		(effects
 			(font
@@
 	(label "xN64_OS_EVENT#"
 		(at 217.17 72.39 180)
+		(fields_autoplaced yes)
 		(effects
 			(font
@@
 	(label "xN64_AD7"
 		(at 217.17 52.07 180)
+		(fields_autoplaced yes)
 		(effects
 			(font
@@
 	(label "xN64_AD6"
 		(at 100.33 77.47 0)
+		(fields_autoplaced yes)
 		(effects
 			(font
@@
 	(label "xN64_AD7"
 		(at 100.33 80.01 0)
+		(fields_autoplaced yes)
 		(effects
 			(font
@@
 	(label "xN64_ALE_H"
 		(at 170.18 69.85 180)
+		(fields_autoplaced yes)
 		(effects
 			(font
@@
 	(label "xN64_S_DAT"
 		(at 217.17 67.31 180)
+		(fields_autoplaced yes)
 		(effects
 			(font
@@
 	(label "xN64_READ#"
 		(at 100.33 110.49 0)
+		(fields_autoplaced yes)
 		(effects
 			(font
@@
 	(label "xN64_ALE_L"
 		(at 100.33 105.41 0)
+		(fields_autoplaced yes)
 		(effects
 			(font
@@
 	(label "xN64_S_CLK"
 		(at 217.17 74.93 180)
+		(fields_autoplaced yes)
 		(effects
 			(font
@@
 	(label "xN64_AD4"
 		(at 100.33 72.39 0)
+		(fields_autoplaced yes)
 		(effects
 			(font
@@
 	(label "xN64_CIC_DATA2"
 		(at 217.17 87.63 180)
+		(fields_autoplaced yes)
 		(effects
 			(font
@@
 	(label "xN64_CIC_DATA1"
 		(at 100.33 133.35 0)
+		(fields_autoplaced yes)
 		(effects
 			(font
@@
 	(label "xN64_AD13"
 		(at 100.33 95.25 0)
+		(fields_autoplaced yes)
 		(effects
 			(font
@@
 	(label "xN64_AD8"
 		(at 100.33 82.55 0)
+		(fields_autoplaced yes)
 		(effects
 			(font
@@
 	(label "xN64_WRITE#"
 		(at 170.18 72.39 180)
+		(fields_autoplaced yes)
 		(effects
 			(font
@@
 	(label "xN64_AD9"
 		(at 217.17 54.61 180)
+		(fields_autoplaced yes)
 		(effects
 			(font
@@
 	(label "xN64_AD0"
 		(at 170.18 39.37 180)
+		(fields_autoplaced yes)
 		(effects
 			(font
@@
 	(label "xN64_AD3"
 		(at 100.33 69.85 0)
+		(fields_autoplaced yes)
 		(effects
 			(font
@@
 	(label "xN64_S_CLK"
 		(at 100.33 120.65 0)
+		(fields_autoplaced yes)
 		(effects
 			(font
@@
 	(label "xN64_AD2"
 		(at 170.18 57.15 180)
+		(fields_autoplaced yes)
 		(effects
 			(font
@@
 	(label "xN64_AD12"
 		(at 170.18 49.53 180)
+		(fields_autoplaced yes)
 		(effects
 			(font
@@
 	(label "xN64_AD1"
 		(at 170.18 34.29 180)
+		(fields_autoplaced yes)
 		(effects
 			(font
@@
 	(label "xN64_AD14"
 		(at 170.18 31.75 180)
+		(fields_autoplaced yes)
 		(effects
 			(font
@@
 	(label "xN64_AD15"
 		(at 100.33 100.33 0)
+		(fields_autoplaced yes)
 		(effects
 			(font
@@
 	(label "xN64_AD11"
 		(at 217.17 36.83 180)
+		(fields_autoplaced yes)
 		(effects
 			(font
@@
 	(label "xN64_ALE_H"
 		(at 100.33 107.95 0)
+		(fields_autoplaced yes)
 		(effects
 			(font
@@
 	(label "xN64_AD15"
 		(at 170.18 36.83 180)
+		(fields_autoplaced yes)
 		(effects
 			(font
@@
 	(label "xN64_AD11"
 		(at 100.33 90.17 0)
+		(fields_autoplaced yes)
 		(effects
 			(font
@@
 	(label "xN64_AD0"
 		(at 100.33 62.23 0)
+		(fields_autoplaced yes)
 		(effects
 			(font
@@
 	(label "xN64_AD14"
 		(at 100.33 97.79 0)
+		(fields_autoplaced yes)
 		(effects
 			(font
@@
 	(label "xN64_WRITE#"
 		(at 100.33 113.03 0)
+		(fields_autoplaced yes)
 		(effects
 			(font
@@
 	(label "xN64_AD9"
 		(at 100.33 85.09 0)
+		(fields_autoplaced yes)
 		(effects
 			(font
@@
 	(label "xN64_AD5"
 		(at 217.17 34.29 180)
+		(fields_autoplaced yes)
 		(effects
 			(font
@@
 	(label "xN64_READ#"
 		(at 170.18 67.31 180)
+		(fields_autoplaced yes)
 		(effects
 			(font
@@
 	(label "xN64_AD5"
 		(at 100.33 74.93 0)
+		(fields_autoplaced yes)
 		(effects
 			(font
@@
 	(label "xN64_AD10"
 		(at 217.17 31.75 180)
+		(fields_autoplaced yes)
 		(effects
 			(font
@@
 	(label "xN64_S_DAT"
 		(at 100.33 118.11 0)
+		(fields_autoplaced yes)
 		(effects
 			(font
@@
 	(label "xN64_CIC_DATA2"
 		(at 100.33 135.89 0)
+		(fields_autoplaced yes)
 		(effects
 			(font
@@
 	(label "xN64_AD13"
 		(at 170.18 54.61 180)
+		(fields_autoplaced yes)
 		(effects
 			(font
@@
 	(label "xN64_AD4"
 		(at 217.17 39.37 180)
+		(fields_autoplaced yes)
 		(effects
 			(font
@@
 		(on_board yes)
 		(dnp no)
-		(property "Reference" "RN4"
+		(property "Reference" "RN1"
 			(at 177.8 26.2382 90)
 			(effects
@@
 		(instances
 			(project "cart-ecp5"
-				(path "/d0de5b81-cadf-4377-8c13-b4d382700369"
-					(reference "RN?")
-					(unit 1)
-				)
 				(path "/d0de5b81-cadf-4377-8c13-b4d382700369/00000000-0000-0000-0000-00005f43b1fd"
 					(reference "RN1")
@@
 		(on_board yes)
 		(dnp no)
-		(property "Reference" "RN6"
+		(property "Reference" "RN2"
 			(at 177.8 44.0182 90)
 			(effects
@@
 		(instances
 			(project "cart-ecp5"
-				(path "/d0de5b81-cadf-4377-8c13-b4d382700369"
-					(reference "RN?")
-					(unit 1)
-				)
 				(path "/d0de5b81-cadf-4377-8c13-b4d382700369/00000000-0000-0000-0000-00005f43b1fd"
 					(reference "RN2")
@@
 		(on_board yes)
 		(dnp no)
-		(property "Reference" "RN8"
+		(property "Reference" "RN3"
 			(at 177.8 61.7982 90)
 			(effects
@@
 		(instances
 			(project "cart-ecp5"
-				(path "/d0de5b81-cadf-4377-8c13-b4d382700369"
-					(reference "RN?")
-					(unit 1)
-				)
 				(path "/d0de5b81-cadf-4377-8c13-b4d382700369/00000000-0000-0000-0000-00005f43b1fd"
 					(reference "RN3")
@@
 		(on_board yes)
 		(dnp no)
-		(property "Reference" "RN5"
+		(property "Reference" "RN4"
 			(at 224.79 26.2382 90)
 			(effects
@@
 		(instances
 			(project "cart-ecp5"
-				(path "/d0de5b81-cadf-4377-8c13-b4d382700369"
-					(reference "RN?")
-					(unit 1)
-				)
 				(path "/d0de5b81-cadf-4377-8c13-b4d382700369/00000000-0000-0000-0000-00005f43b1fd"
 					(reference "RN4")
@@
 		(on_board yes)
 		(dnp no)
-		(property "Reference" "RN7"
+		(property "Reference" "RN5"
 			(at 224.79 44.0182 90)
 			(effects
@@
 		(instances
 			(project "cart-ecp5"
-				(path "/d0de5b81-cadf-4377-8c13-b4d382700369"
-					(reference "RN?")
-					(unit 1)
-				)
 				(path "/d0de5b81-cadf-4377-8c13-b4d382700369/00000000-0000-0000-0000-00005f43b1fd"
 					(reference "RN5")
@@
 		(on_board yes)
 		(dnp no)
-		(property "Reference" "RN9"
+		(property "Reference" "RN6"
 			(at 224.79 61.7982 90)
 			(effects
@@
 		(instances
 			(project "cart-ecp5"
-				(path "/d0de5b81-cadf-4377-8c13-b4d382700369"
-					(reference "RN?")
-					(unit 1)
-				)
 				(path "/d0de5b81-cadf-4377-8c13-b4d382700369/00000000-0000-0000-0000-00005f43b1fd"
 					(reference "RN6")
@@
 		(on_board yes)
 		(dnp no)
-		(property "Reference" "RN?"
+		(property "Reference" "RN8"
 			(at 224.79 79.5782 90)
 			(effects
@@
 		(instances
 			(project "cart-ecp5"
-				(path "/d0de5b81-cadf-4377-8c13-b4d382700369"
-					(reference "RN?")
-					(unit 1)
-				)
 				(path "/d0de5b81-cadf-4377-8c13-b4d382700369/00000000-0000-0000-0000-00005f43b1fd"
 					(reference "RN8")
@@
 					(unit 1)
 				)
-				(path "/d0de5b81-cadf-4377-8c13-b4d382700369/00000000-0000-0000-0000-00005f3e46de"
-					(reference "C?")
-					(unit 1)
-				)
 			)
 		)
@@
 					(unit 1)
 				)
-				(path "/d0de5b81-cadf-4377-8c13-b4d382700369/00000000-0000-0000-0000-00005f3e46de"
-					(reference "#PWR?")
-					(unit 1)
-				)

Commit message: hardware: Substitute library symbol for ATtiny microcontroller
Parts:
- U4: footprint Package_SO:SOIJ-8_5.3x5.3mm_P1.27mm -> Package_SO:SOIC-8W_5.3x5.3mm_P1.27mm; symbol cart-ecp5-rescue:ATtiny25-20SU-MCU_Microchip_ATtiny -> MCU_Microchip_ATtiny:ATtiny45-20S
Changed lines of the file:
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@@
 	)
 	(symbol
-		(lib_id "cart-ecp5-rescue:ATtiny25-20SU-MCU_Microchip_ATtiny")
+		(lib_id "MCU_Microchip_ATtiny:ATtiny45-20S")
 		(at 205.74 125.73 0)
 		(mirror y)
@@
 			)
 		)
-		(property "Footprint" "Package_SO:SOIJ-8_5.3x5.3mm_P1.27mm"
+		(property "Footprint" "Package_SO:SOIC-8W_5.3x5.3mm_P1.27mm"
 			(at 205.74 125.73 0)
 			(effects
@@
 			)
 		)
-		(property "Description" ""
+		(property "Description" "20MHz, 4kB Flash, 256B SRAM, 256B EEPROM, debugWIRE, SOIC-8W"
 			(at 205.74 125.73 0)
 			(effects
@@
 		)
 		(pin "1"
+		)
+		(instances
+			(project "cart-ecp5"
+				(path "/d0de5b81-cadf-4377-8c13-b4d382700369/00000000-0000-0000-0000-00005f43b1fd"
+					(reference "#PWR013")
+					(unit 1)
+				)
+			)
 		)
 	)
@@
 		(pin "1"
 		)
+		(instances
+			(project "cart-ecp5"
+				(path "/d0de5b81-cadf-4377-8c13-b4d382700369/00000000-0000-0000-0000-00005f43b1fd"
+					(reference "#PWR015")
+					(unit 1)
+				)
+			)
+		)
 	)
 	(symbol
@@
 		(pin "1"
 		)
-	)
+		(instances
+			(project "cart-ecp5"
+				(path "/d0de5b81-cadf-4377-8c13-b4d382700369/00000000-0000-0000-0000-00005f43b1fd"
+					(reference "#PWR014")
+					(unit 1)
+				)
+			)
+		)
+	)
